File: sign.sch (KiCad schematic (older format))
At the start: 148 parts, among them J1 CONN_01X02, J2 CONN_01X02, J3 CONN_01X02, J4 CONN_01X02, J5 CONN_01X02, J6 CONN_01X02, J7 CONN_01X02, J8 CONN_01X02, J9 CONN_01X02, U1 APA102C_x6, U10 APA102C_x2, U100 APA102C_x6, U101 APA102C_x4, U102 APA102C_x2, U103 APA102C_x1, U104 APA102C_x3, U105 APA102C_x5, U106 APA102C_x2, U107 APA102C_x3, U108 APA102C_x10, U109 APA102C_x9, U11 APA102C_x2, U110 APA102C_x3, U111 APA102C_x12, U112 APA102C_x16, U113 APA102C_x8, U114 APA102C_x13, U115 APA102C_x3, U116 APA102C_x6, U117 APA102C_x3, U118 APA102C_x6, U119 APA102C_x3, U12 APA102C_x2, U120 APA102C_x2, U121 APA102C_x6, U122 APA102C_x3, U123 APA102C_x6, U124 APA102C_x7, U125 APA102C_x12, U126 APA102C_x6, U127 APA102C_x11, U128 APA102C_x4, U129 APA102C_x6, U13 APA102C_x2, U130 APA102C_x2, U131 APA102C_x2, U132 APA102C_x3, U133 APA102C_x1, U134 APA102C_x3, U135 APA102C_x3, U136 APA102C_x12, U137 APA102C_x12, U138 APA102C_x9, U139 APA102C_x4, U14 APA102C_x3, U15 APA102C_x3, U16 APA102C_x3, U17 APA102C_x3, U18 APA102C_x5, U19 APA102C_x6, U2 APA102C_x8, U20 APA102C_x2, U21 APA102C_x7, U22 APA102C_x5, U23 APA102C_x7, U24 APA102C_x3, U25 APA102C_x2, U26 APA102C_x7, U27 APA102C_x2, U28 APA102C_x3, U29 APA102C_x5, U3 APA102C_x11, U30 APA102C_x2, U31 APA102C_x5, U32 APA102C_x2, U33 APA102C_x8, U34 APA102C_x9, U35 APA102C_x3, U36 APA102C_x2, U37 APA102C_x5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

Commit message: Wire all the letters!
Parts:
- added J10, J11, J12, J13, J14, J15, J16, J17, J18, J19, J20, J21, J22, J23, J24, J25, J26, J27, J28, J29, J30: CONN_01X02, Pin_Headers:Pin_Header_Straight_1x02, symbol CONN_01X02
Connections:
- net +5V: now also U102.4 (Vin), U36.4 (Vin), U54.4 (Vin), U71.4 (Vin), U81.4 (Vin), U92.4 (Vin), U98.4 (Vin), J10.2 (P2), J13.2 (P2), J15.2 (P2), J17.2 (P2), J21.2 (P2), J23.2 (P2), J25.2 (P2)
- net GND: now also U102.1 (Gin), U36.1 (Gin), U54.1 (Gin), U71.1 (Gin), U81.1 (Gin), U92.1 (Gin), U98.1 (Gin), J10.1 (P1), J13.1 (P1), J15.1 (P1), J17.1 (P1), J21.1 (P1), J23.1 (P1), J25.1 (P1)
- net at U18.1 (Gin): now also U21.5 (Gout)
- net at U18.2 (Cin): now also U21.6 (Cout)
- net at U18.3 (Din): now also U21.7 (Dout)
- net at U18.4 (Vin): now also U21.8 (Vout)
- net at U18.5 (Gout): now also U23.1 (Gin)
- net at U18.6 (Cout): now also U23.2 (Cin)
- net at U18.7 (Dout): now also U23.3 (Din)
- net at U18.8 (Vout): now also U23.4 (Vin)
- net at U21.1 (Gin): now also U24.5 (Gout)
- net at U21.2 (Cin): now also U24.6 (Cout)
- net at U21.3 (Din): now also U24.7 (Dout)
- net at U21.4 (Vin): now also U24.8 (Vout)
- net at U23.6 (Cout): now also J12.1 (P1)
- net at U23.7 (Dout): now also J12.2 (P2)
- net at U24.1 (Gin): now also U27.5 (Gout)
- net at U24.2 (Cin): now also U27.6 (Cout)
- net at U24.3 (Din): now also U27.7 (Dout)
- net at U24.4 (Vin): now also U27.8 (Vout)
- net at U26.1 (Gin): now also U28.5 (Gout)
- net at U26.2 (Cin): now also U28.6 (Cout)
- net at U26.3 (Din): now also U28.7 (Dout)
- net at U26.4 (Vin): now also U28.8 (Vout)
- net at U26.5 (Gout): now also U29.1 (Gin)
- net at U26.6 (Cout): now also U29.2 (Cin)
- net at U26.7 (Dout): now also U29.3 (Din)
- net at U26.8 (Vout): now also U29.4 (Vin)
- net at U27.1 (Gin): now also U30.5 (Gout)
- net at U27.2 (Cin): now also U30.6 (Cout)
- net at U27.3 (Din): now also U30.7 (Dout)
- net at U27.4 (Vin): now also U30.8 (Vout)
- net at U28.1 (Gin): now also U32.5 (Gout)
- net at U28.2 (Cin): now also U32.6 (Cout)
- net at U28.3 (Din): now also U32.7 (Dout)
- net at U28.4 (Vin): now also U32.8 (Vout)
- net at U29.5 (Gout): now also U33.1 (Gin)
- net at U29.6 (Cout): now also U33.2 (Cin)
- net at U29.7 (Dout): now also U33.3 (Din)
- net at U29.8 (Vout): now also U33.4 (Vin)
- net at U30.1 (Gin): now also U48.5 (Gout)
- net at U30.2 (Cin): now also U48.6 (Cout)
- net at U30.3 (Din): now also U48.7 (Dout)
- net at U30.4 (Vin): now also U48.8 (Vout)
- net at U32.1 (Gin): now also U35.5 (Gout)
- net at U32.2 (Cin): now also U35.6 (Cout)
- net at U32.3 (Din): now also U35.7 (Dout)
- net at U32.4 (Vin): now also U35.8 (Vout)
- net at U33.5 (Gout): now also U37.1 (Gin)
- net at U33.6 (Cout): now also U37.2 (Cin)
- net at U33.7 (Dout): now also U37.3 (Din)
- net at U33.8 (Vout): now also U37.4 (Vin)
- net at U35.1 (Gin): now also U43.5 (Gout)
- net at U35.2 (Cin): now also U43.6 (Cout)
- net at U35.3 (Din): now also U43.7 (Dout)
- net at U35.4 (Vin): now also U43.8 (Vout)
- net at U36.2 (Cin): now also J11.1 (P1)
- net at U36.3 (Din): now also J11.2 (P2)
- net at U36.5 (Gout): now also U39.1 (Gin)
- net at U36.6 (Cout): now also U39.2 (Cin)
- net at U36.7 (Dout): now also U39.3 (Din)
- net at U36.8 (Vout): now also U39.4 (Vin)
- net at U37.5 (Gout): now also U40.1 (Gin)
- net at U37.6 (Cout): now also U40.2 (Cin)
- net at U37.7 (Dout): now also U40.3 (Din)
- net at U37.8 (Vout): now also U40.4 (Vin)
- net at U39.5 (Gout): now also U43.1 (Gin)
- net at U39.6 (Cout): now also U43.2 (Cin)
- net at U39.7 (Dout): now also U43.3 (Din)
- net at U39.8 (Vout): now also U43.4 (Vin)
- net at U40.5 (Gout): now also U44.1 (Gin)
- net at U40.6 (Cout): now also U44.2 (Cin)
- net at U40.7 (Dout): now also U44.3 (Din)
- net at U40.8 (Vout): now also U44.4 (Vin)
- net at U44.5 (Gout): now also U51.4 (Vin)
- net at U44.6 (Cout): now also U51.3 (Din)
- net at U44.7 (Dout): now also U51.2 (Cin)
- net at U44.8 (Vout): now also U51.1 (Gin)
- net at U47.1 (Gin): now also U51.5 (Gout)
- net at U47.2 (Cin): now also U51.6 (Cout)
- net at U47.3 (Din): now also U51.7 (Dout)
- net at U47.4 (Vin): now also U51.8 (Vout)
- net at U47.5 (Gout): now also U48.1 (Gin)
- net at U47.6 (Cout): now also U48.2 (Cin)
- net at U47.7 (Dout): now also U48.3 (Din)
- net at U47.8 (Vout): now also U48.4 (Vin)
- net at U54.2 (Cin): now also J14.1 (P1)
- net at U54.3 (Din): now also J14.2 (P2)
- net at U71.2 (Cin): now also J16.1 (P1)
- net at U71.3 (Din): now also J16.2 (P2)
- net at U75.6 (Cout): now also J19.1 (P1)
- net at U75.7 (Dout): now also J19.2 (P2)
- net at U78.6 (Cout): now also J20.1 (P1)
- net at U78.7 (Dout): now also J20.2 (P2)
- net at U81.2 (Cin): now also J18.1 (P1)
- net at U81.3 (Din): now also J18.2 (P2)
- net at U92.2 (Cin): now also J22.1 (P1)
- net at U92.3 (Din): now also J22.2 (P2)
- net at U96.6 (Cout): now also J27.1 (P1)
- net at U96.7 (Dout): now also J27.2 (P2)
- net at U98.2 (Cin): now also J24.1 (P1)
- net at U98.3 (Din): now also J24.2 (P2)
- net at U98.5 (Gout): now also U101.1 (Gin)
- net at U98.6 (Cout): now also U101.2 (Cin)
- net at U98.7 (Dout): now also U101.3 (Din)
- net at U98.8 (Vout): now also U101.4 (Vin)
- net at U99.6 (Cout): now also J28.1 (P1)
- net at U99.7 (Dout): now also J28.2 (P2)
- net at U101.5 (Gout): now also U104.1 (Gin)
- net at U101.6 (Cout): now also U104.2 (Cin)
- net at U101.7 (Dout): now also U104.3 (Din)
- net at U101.8 (Vout): now also U104.4 (Vin)
- net at U102.2 (Cin): now also J26.1 (P1)
- net at U102.3 (Din): now also J26.2 (P2)
- net at U102.5 (Gout): now also U105.1 (Gin)
- net at U102.6 (Cout): now also U105.2 (Cin)
- net at U102.7 (Dout): now also U105.3 (Din)
- net at U102.8 (Vout): now also U105.4 (Vin)
- net at U104.5 (Gout): now also U107.1 (Gin)
- net at U104.6 (Cout): now also U107.2 (Cin)
- net at U104.7 (Dout): now also U107.3 (Din)
- net at U104.8 (Vout): now also U107.4 (Vin)
- net at U105.5 (Gout): now also U108.1 (Gin)
- net at U105.6 (Cout): now also U108.2 (Cin)
- net at U105.7 (Dout): now also U108.3 (Din)
- net at U105.8 (Vout): now also U108.4 (Vin)
- net at U106.1 (Gin): now also U109.5 (Gout)
- net at U106.2 (Cin): now also U109.6 (Cout)
- net at U106.3 (Din): now also U109.7 (Dout)
- net at U106.4 (Vin): now also U109.8 (Vout)
- net at U106.6 (Cout): now also J29.1 (P1)
- net at U106.7 (Dout): now also J29.2 (P2)
- net at U107.5 (Gout): now also U110.1 (Gin)
- net at U107.6 (Cout): now also U110.2 (Cin)
- net at U107.7 (Dout): now also U110.3 (Din)
- net at U107.8 (Vout): now also U110.4 (Vin)
- net at U108.5 (Gout): now also U111.1 (Gin)
- net at U108.6 (Cout): now also U111.2 (Cin)
- net at U108.7 (Dout): now also U111.3 (Din)
- net at U108.8 (Vout): now also U111.4 (Vin)
- net at U109.1 (Gin): now also U130.5 (Gout)
- net at U109.2 (Cin): now also U130.6 (Cout)
- net at U109.3 (Din): now also U130.7 (Dout)
- net at U109.4 (Vin): now also U130.8 (Vout)
- net at U110.5 (Gout): now also U112.1 (Gin)
- net at U110.6 (Cout): now also U112.2 (Cin)
- net at U110.7 (Dout): now also U112.3 (Din)
- net at U110.8 (Vout): now also U112.4 (Vin)
- net at U111.5 (Gout): now also U113.1 (Gin)
- net at U111.6 (Cout): now also U113.2 (Cin)
- net at U111.7 (Dout): now also U113.3 (Din)
- net at U111.8 (Vout): now also U113.4 (Vin)
- net at U112.5 (Gout): now also U114.1 (Gin)
- net at U112.6 (Cout): now also U114.2 (Cin)
- net at U112.7 (Dout): now also U114.3 (Din)
- net at U112.8 (Vout): now also U114.4 (Vin)
- net at U113.5 (Gout): now also U115.1 (Gin)
- net at U113.6 (Cout): now also U115.2 (Cin)
- net at U113.7 (Dout): now also U115.3 (Din)
- net at U113.8 (Vout): now also U115.4 (Vin)
- net at U114.5 (Gout): now also U116.1 (Gin)
- net at U114.6 (Cout): now also U116.2 (Cin)
- net at U114.7 (Dout): now also U116.3 (Din)
- net at U114.8 (Vout): now also U116.4 (Vin)
- net at U115.5 (Gout): now also U117.1 (Gin)
- net at U115.6 (Cout): now also U117.2 (Cin)
- net at U115.7 (Dout): now also U117.3 (Din)
- net at U115.8 (Vout): now also U117.4 (Vin)
- net at U116.5 (Gout): now also U118.1 (Gin)
- net at U116.6 (Cout): now also U118.2 (Cin)
- net at U116.7 (Dout): now also U118.3 (Din)
- net at U116.8 (Vout): now also U118.4 (Vin)
- net at U117.5 (Gout): now also U119.1 (Gin)
- net at U117.6 (Cout): now also U119.2 (Cin)
- net at U117.7 (Dout): now also U119.3 (Din)
- net at U117.8 (Vout): now also U119.4 (Vin)
- net at U118.5 (Gout): now also U121.1 (Gin)
- net at U118.6 (Cout): now also U121.2 (Cin)
- net at U118.7 (Dout): now also U121.3 (Din)
- net at U118.8 (Vout): now also U121.4 (Vin)
- net at U119.5 (Gout): now also U122.1 (Gin)
- net at U119.6 (Cout): now also U122.2 (Cin)
- net at U119.7 (Dout): now also U122.3 (Din)
- net at U119.8 (Vout): now also U122.4 (Vin)
- net at U120.1 (Gin): now also U123.5 (Gout)
- net at U120.2 (Cin): now also U123.6 (Cout)
- net at U120.3 (Din): now also U123.7 (Dout)
- net at U120.4 (Vin): now also U123.8 (Vout)
- net at U120.5 (Gout): now also U125.1 (Gin)
- net at U120.6 (Cout): now also U125.2 (Cin)
- net at U120.7 (Dout): now also U125.3 (Din)
- net at U120.8 (Vout): now also U125.4 (Vin)
- net at U121.5 (Gout): now also U124.1 (Gin)
- net at U121.6 (Cout): now also U124.2 (Cin)
- net at U121.7 (Dout): now also U124.3 (Din)
- net at U121.8 (Vout): now also U124.4 (Vin)
- net at U122.5 (Gout): now also U123.1 (Gin)
- net at U122.6 (Cout): now also U123.2 (Cin)
- net at U122.7 (Dout): now also U123.3 (Din)
- net at U122.8 (Vout): now also U123.4 (Vin)
- net at U124.5 (Gout): now also U126.1 (Gin)
- net at U124.6 (Cout): now also U126.2 (Cin)
- net at U124.7 (Dout): now also U126.3 (Din)
- net at U124.8 (Vout): now also U126.4 (Vin)
- net at U125.5 (Gout): now also U127.1 (Gin)
- net at U125.6 (Cout): now also U127.2 (Cin)
- net at U125.7 (Dout): now also U127.3 (Din)
- net at U125.8 (Vout): now also U127.4 (Vin)
- net at U126.5 (Gout): now also U128.1 (Gin)
- net at U126.6 (Cout): now also U128.2 (Cin)
- net at U126.7 (Dout): now also U128.3 (Din)
- net at U126.8 (Vout): now also U128.4 (Vin)
- net at U127.5 (Gout): now also U129.1 (Gin)
- net at U127.6 (Cout): now also U129.2 (Cin)
- net at U127.7 (Dout): now also U129.3 (Din)
- net at U127.8 (Vout): now also U129.4 (Vin)
- net at U128.5 (Gout): now also U130.1 (Gin)
- net at U128.6 (Cout): now also U130.2 (Cin)
- net at U128.7 (Dout): now also U130.3 (Din)
- net at U128.8 (Vout): now also U130.4 (Vin)
- net at U129.5 (Gout): now also U131.1 (Gin)
- net at U129.6 (Cout): now also U131.2 (Cin)
- net at U129.7 (Dout): now also U131.3 (Din)
- net at U129.8 (Vout): now also U131.4 (Vin)
- net at U131.5 (Gout): now also U132.1 (Gin)
- net at U131.6 (Cout): now also U132.2 (Cin)
- net at U131.7 (Dout): now also U132.3 (Din)
- net at U131.8 (Vout): now also U132.4 (Vin)
- net at U132.5 (Gout): now also U134.1 (Gin)
- net at U132.6 (Cout): now also U134.2 (Cin)
- net at U132.7 (Dout): now also U134.3 (Din)
- net at U132.8 (Vout): now also U134.4 (Vin)
- net at U133.1 (Gin): now also U135.5 (Gout)
- net at U133.2 (Cin): now also U135.6 (Cout)
- net at U133.3 (Din): now also U135.7 (Dout)
- net at U133.4 (Vin): now also U135.8 (Vout)
- net at U133.5 (Gout): now also U136.1 (Gin)
- net at U133.6 (Cout): now also U136.2 (Cin)
- net at U133.7 (Dout): now also U136.3 (Din)
- net at U133.8 (Vout): now also U136.4 (Vin)
- net at U134.5 (Gout): now also U135.1 (Gin)
- net at U134.6 (Cout): now also U135.2 (Cin)
- net at U134.7 (Dout): now also U135.3 (Din)
- net at U134.8 (Vout): now also U135.4 (Vin)
- net at U136.5 (Gout): now also U137.1 (Gin)
- net at U136.6 (Cout): now also U137.2 (Cin)
- net at U136.7 (Dout): now also U137.3 (Din)
- net at U136.8 (Vout): now also U137.4 (Vin)
- net at U137.5 (Gout): now also U138.1 (Gin)
- net at U137.6 (Cout): now also U138.2 (Cin)
- net at U137.7 (Dout): now also U138.3 (Din)
- net at U137.8 (Vout): now also U138.4 (Vin)
- net at U138.5 (Gout): now also U139.1 (Gin)
- net at U138.6 (Cout): now also U139.2 (Cin)
- net at U138.7 (Dout): now also U139.3 (Din)
- net at U138.8 (Vout): now also U139.4 (Vin)
- net at U139.6 (Cout): now also J30.1 (P1)
- net at U139.7 (Dout): now also J30.2 (P2)
- no-connect marks 2 -> 20

Commit message: Untangle all the pcb letters and wire up both d's.
Parts:
- J1, J10, J11, J12, J13, J14, J15, J16, J17, J18, J19, J2, J20, J21, J22, J23, J24, J25, J26, J27, J28, J29, J3, J30, J4, J5, J6, J7, J8, J9: footprint Pin_Headers:Pin_Header_Straight_1x02 -> Pin_Headers:Pin_Header_Straight_1x02_Pitch2.54mm
Changed lines of the file:
@@
 F 0 "J1" H 1400 7200 50  0000 C CNN
 F 1 "CONN_01X02" V 1500 7050 50  0000 C CNN
-F 2 "Pin_Headers:Pin_Header_Straight_1x02" H 1400 7050 50  0001 C CNN
+F 2 "Pin_Headers:Pin_Header_Straight_1x02_Pitch2.54mm" H 1400 7050 50  0001 C CNN
 F 3 "" H 1400 7050 50  0001 C CNN
 	1    1400 7050
@@
 F 0 "J2" H 1400 7550 50  0000 C CNN
 F 1 "CONN_01X02" V 1500 7400 50  0000 C CNN
-F 2 "Pin_Headers:Pin_Header_Straight_1x02" H 1400 7400 50  0001 C CNN
+F 2 "Pin_Headers:Pin_Header_Straight_1x02_Pitch2.54mm" H 1400 7400 50  0001 C CNN
 F 3 "" H 1400 7400 50  0001 C CNN
 	1    1400 7400
@@
 F 0 "J3" H 1400 7900 50  0000 C CNN
 F 1 "CONN_01X02" V 1500 7750 50  0000 C CNN
-F 2 "Pin_Headers:Pin_Header_Straight_1x02" H 1400 7750 50  0001 C CNN
+F 2 "Pin_Headers:Pin_Header_Straight_1x02_Pitch2.54mm" H 1400 7750 50  0001 C CNN
 F 3 "" H 1400 7750 50  0001 C CNN
 	1    1400 7750
@@
 F 0 "J4" H 8450 7900 50  0000 C CNN
 F 1 "CONN_01X02" V 8550 7750 50  0000 C CNN
-F 2 "Pin_Headers:Pin_Header_Straight_1x02" H 8450 7750 50  0001 C CNN
+F 2 "Pin_Headers:Pin_Header_Straight_1x02_Pitch2.54mm" H 8450 7750 50  0001 C CNN
 F 3 "" H 8450 7750 50  0001 C CNN
 	1    8450 7750
@@
 F 0 "J5" H 8450 8250 50  0000 C CNN
 F 1 "CONN_01X02" V 8550 8100 50  0000 C CNN
-F 2 "Pin_Headers:Pin_Header_Straight_1x02" H 8450 8100 50  0001 C CNN
+F 2 "Pin_Headers:Pin_Header_Straight_1x02_Pitch2.54mm" H 8450 8100 50  0001 C CNN
 F 3 "" H 8450 8100 50  0001 C CNN
 	1    8450 8100
@@
 F 0 "J6" H 8450 8600 50  0000 C CNN
 F 1 "CONN_01X02" V 8550 8450 50  0000 C CNN
-F 2 "Pin_Headers:Pin_Header_Straight_1x02" H 8450 8450 50  0001 C CNN
+F 2 "Pin_Headers:Pin_Header_Straight_1x02_Pitch2.54mm" H 8450 8450 50  0001 C CNN
 F 3 "" H 8450 8450 50  0001 C CNN
 	1    8450 8450
@@
 F 0 "J7" H 16250 7900 50  0000 C CNN
 F 1 "CONN_01X02" V 16350 7750 50  0000 C CNN
-F 2 "Pin_Headers:Pin_Header_Straight_1x02" H 16250 7750 50  0001 C CNN
+F 2 "Pin_Headers:Pin_Header_Straight_1x02_Pitch2.54mm" H 16250 7750 50  0001 C CNN
 F 3 "" H 16250 7750 50  0001 C CNN
 	1    16250 7750
@@
 F 0 "J8" H 16250 8250 50  0000 C CNN
 F 1 "CONN_01X02" V 16350 8100 50  0000 C CNN
-F 2 "Pin_Headers:Pin_Header_Straight_1x02" H 16250 8100 50  0001 C CNN
+F 2 "Pin_Headers:Pin_Header_Straight_1x02_Pitch2.54mm" H 16250 8100 50  0001 C CNN
 F 3 "" H 16250 8100 50  0001 C CNN
 	1    16250 8100
@@
 F 0 "J9" H 16250 8600 50  0000 C CNN
 F 1 "CONN_01X02" V 16350 8450 50  0000 C CNN
-F 2 "Pin_Headers:Pin_Header_Straight_1x02" H 16250 8450 50  0001 C CNN
+F 2 "Pin_Headers:Pin_Header_Straight_1x02_Pitch2.54mm" H 16250 8450 50  0001 C CNN
 F 3 "" H 16250 8450 50  0001 C CNN
 	1    16250 8450
@@
 F 0 "J23" H 22250 12800 50  0000 C CNN
 F 1 "CONN_01X02" V 22350 12650 50  0000 C CNN
-F 2 "Pin_Headers:Pin_Header_Straight_1x02" H 22250 12650 50  0001 C CNN
+F 2 "Pin_Headers:Pin_Header_Straight_1x02_Pitch2.54mm" H 22250 12650 50  0001 C CNN
 F 3 "" H 22250 12650 50  0001 C CNN
 	1    22250 12650
@@
 F 0 "J24" H 22250 13150 50  0000 C CNN
 F 1 "CONN_01X02" V 22350 13000 50  0000 C CNN
-F 2 "Pin_Headers:Pin_Header_Straight_1x02" H 22250 13000 50  0001 C CNN
+F 2 "Pin_Headers:Pin_Header_Straight_1x02_Pitch2.54mm" H 22250 13000 50  0001 C CNN
 F 3 "" H 22250 13000 50  0001 C CNN
 	1    22250 13000
@@
 F 0 "J29" H 24700 4450 50  0000 C CNN
 F 1 "CONN_01X02" V 24800 4300 50  0000 C CNN
-F 2 "Pin_Headers:Pin_Header_Straight_1x02" H 24700 4300 50  0001 C CNN
+F 2 "Pin_Headers:Pin_Header_Straight_1x02_Pitch2.54mm" H 24700 4300 50  0001 C CNN
 F 3 "" H 24700 4300 50  0001 C CNN
 	1    24700 4300
@@
 F 0 "J15" H 16850 16900 50  0000 C CNN
 F 1 "CONN_01X02" V 16950 16750 50  0000 C CNN
-F 2 "Pin_Headers:Pin_Header_Straight_1x02" H 16850 16750 50  0001 C CNN
+F 2 "Pin_Headers:Pin_Header_Straight_1x02_Pitch2.54mm" H 16850 16750 50  0001 C CNN
 F 3 "" H 16850 16750 50  0001 C CNN
 	1    16850 16750
@@
 F 0 "J16" H 16850 17250 50  0000 C CNN
 F 1 "CONN_01X02" V 16950 17100 50  0000 C CNN
-F 2 "Pin_Headers:Pin_Header_Straight_1x02" H 16850 17100 50  0001 C CNN
+F 2 "Pin_Headers:Pin_Header_Straight_1x02_Pitch2.54mm" H 16850 17100 50  0001 C CNN
 F 3 "" H 16850 17100 50  0001 C CNN
 	1    16850 17100
@@
 F 0 "J20" H 19350 16550 50  0000 C CNN
 F 1 "CONN_01X02" V 19450 16400 50  0000 C CNN
-F 2 "Pin_Headers:Pin_Header_Straight_1x02" H 19350 16400 50  0001 C CNN
+F 2 "Pin_Headers:Pin_Header_Straight_1x02_Pitch2.54mm" H 19350 16400 50  0001 C CNN
 F 3 "" H 19350 16400 50  0001 C CNN
 	1    19350 16400
@@
 F 0 "J21" H 21050 16900 50  0000 C CNN
 F 1 "CONN_01X02" V 21150 16750 50  0000 C CNN
-F 2 "Pin_Headers:Pin_Header_Straight_1x02" H 21050 16750 50  0001 C CNN
+F 2 "Pin_Headers:Pin_Header_Straight_1x02_Pitch2.54mm" H 21050 16750 50  0001 C CNN
 F 3 "" H 21050 16750 50  0001 C CNN
 	1    21050 16750
@@
 F 0 "J22" H 21050 17250 50  0000 C CNN
 F 1 "CONN_01X02" V 21150 17100 50  0000 C CNN
-F 2 "Pin_Headers:Pin_Header_Straight_1x02" H 21050 17100 50  0001 C CNN
+F 2 "Pin_Headers:Pin_Header_Straight_1x02_Pitch2.54mm" H 21050 17100 50  0001 C CNN
 F 3 "" H 21050 17100 50  0001 C CNN
 	1    21050 17100
@@
 F 0 "J28" H 23550 16550 50  0000 C CNN
 F 1 "CONN_01X02" V 23650 16400 50  0000 C CNN
-F 2 "Pin_Headers:Pin_Header_Straight_1x02" H 23550 16400 50  0001 C CNN
+F 2 "Pin_Headers:Pin_Header_Straight_1x02_Pitch2.54mm" H 23550 16400 50  0001 C CNN
 F 3 "" H 23550 16400 50  0001 C CNN
 	1    23550 16400
@@
 F 0 "J13" H 12050 27200 50  0000 C CNN
 F 1 "CONN_01X02" V 12150 27050 50  0000 C CNN
-F 2 "Pin_Headers:Pin_Header_Straight_1x02" H 12050 27050 50  0001 C CNN
+F 2 "Pin_Headers:Pin_Header_Straight_1x02_Pitch2.54mm" H 12050 27050 50  0001 C CNN
 F 3 "" H 12050 27050 50  0001 C CNN
 	1    12050 27050
@@
 F 0 "J14" H 12050 27550 50  0000 C CNN
 F 1 "CONN_01X02" V 12150 27400 50  0000 C CNN
-F 2 "Pin_Headers:Pin_Header_Straight_1x02" H 12050 27400 50  0001 C CNN
+F 2 "Pin_Headers:Pin_Header_Straight_1x02_Pitch2.54mm" H 12050 27400 50  0001 C CNN
 F 3 "" H 12050 27400 50  0001 C CNN
 	1    12050 27400
@@
 F 0 "J25" H 22850 25300 50  0000 C CNN
 F 1 "CONN_01X02" V 22950 25150 50  0000 C CNN
-F 2 "Pin_Headers:Pin_Header_Straight_1x02" H 22850 25150 50  0001 C CNN
+F 2 "Pin_Headers:Pin_Header_Straight_1x02_Pitch2.54mm" H 22850 25150 50  0001 C CNN
 F 3 "" H 22850 25150 50  0001 C CNN
 	1    22850 25150
@@
 F 0 "J26" H 22850 25650 50  0000 C CNN
 F 1 "CONN_01X02" V 22950 25500 50  0000 C CNN
-F 2 "Pin_Headers:Pin_Header_Straight_1x02" H 22850 25500 50  0001 C CNN
+F 2 "Pin_Headers:Pin_Header_Straight_1x02_Pitch2.54mm" H 22850 25500 50  0001 C CNN
 F 3 "" H 22850 25500 50  0001 C CNN
 	1    22850 25500
@@
 F 0 "J17" H 18650 25350 50  0000 C CNN
 F 1 "CONN_01X02" V 18750 25200 50  0000 C CNN
-F 2 "Pin_Headers:Pin_Header_Straight_1x02" H 18650 25200 50  0001 C CNN
+F 2 "Pin_Headers:Pin_Header_Straight_1x02_Pitch2.54mm" H 18650 25200 50  0001 C CNN
 F 3 "" H 18650 25200 50  0001 C CNN
 	1    18650 25200
@@
 F 0 "J18" H 18650 25700 50  0000 C CNN
 F 1 "CONN_01X02" V 18750 25550 50  0000 C CNN
-F 2 "Pin_Headers:Pin_Header_Straight_1x02" H 18650 25550 50  0001 C CNN
+F 2 "Pin_Headers:Pin_Header_Straight_1x02_Pitch2.54mm" H 18650 25550 50  0001 C CNN
 F 3 "" H 18650 25550 50  0001 C CNN
 	1    18650 25550
@@
 F 0 "J10" H 5450 17400 50  0000 C CNN
 F 1 "CONN_01X02" V 5550 17250 50  0000 C CNN
-F 2 "Pin_Headers:Pin_Header_Straight_1x02" H 5450 17250 50  0001 C CNN
+F 2 "Pin_Headers:Pin_Header_Straight_1x02_Pitch2.54mm" H 5450 17250 50  0001 C CNN
 F 3 "" H 5450 17250 50  0001 C CNN
 	1    5450 17250
@@
 F 0 "J11" H 5450 17750 50  0000 C CNN
 F 1 "CONN_01X02" V 5550 17600 50  0000 C CNN
-F 2 "Pin_Headers:Pin_Header_Straight_1x02" H 5450 17600 50  0001 C CNN
+F 2 "Pin_Headers:Pin_Header_Straight_1x02_Pitch2.54mm" H 5450 17600 50  0001 C CNN
 F 3 "" H 5450 17600 50  0001 C CNN
 	1    5450 17600
@@
 F 0 "J19" H 18900 19050 50  0000 C CNN
 F 1 "CONN_01X02" V 19000 18900 50  0000 C CNN
-F 2 "Pin_Headers:Pin_Header_Straight_1x02" H 18900 18900 50  0001 C CNN
+F 2 "Pin_Headers:Pin_Header_Straight_1x02_Pitch2.54mm" H 18900 18900 50  0001 C CNN
 F 3 "" H 18900 18900 50  0001 C CNN
 	1    18900 18900
@@
 F 0 "J27" H 23100 19100 50  0000 C CNN
 F 1 "CONN_01X02" V 23200 18950 50  0000 C CNN
-F 2 "Pin_Headers:Pin_Header_Straight_1x02" H 23100 18950 50  0001 C CNN
+F 2 "Pin_Headers:Pin_Header_Straight_1x02_Pitch2.54mm" H 23100 18950 50  0001 C CNN
 F 3 "" H 23100 18950 50  0001 C CNN
 	1    23100 18950
@@
 F 0 "J30" H 34500 23300 50  0000 C CNN
 F 1 "CONN_01X02" V 34600 23150 50  0000 C CNN
-F 2 "Pin_Headers:Pin_Header_Straight_1x02" H 34500 23150 50  0001 C CNN
+F 2 "Pin_Headers:Pin_Header_Straight_1x02_Pitch2.54mm" H 34500 23150 50  0001 C CNN
 F 3 "" H 34500 23150 50  0001 C CNN
 	1    34500 23150
@@
 F 0 "J12" H 6550 16450 50  0000 C CNN
 F 1 "CONN_01X02" V 6650 16300 50  0000 C CNN
-F 2 "Pin_Headers:Pin_Header_Straight_1x02" H 6550 16300 50  0001 C CNN
+F 2 "Pin_Headers:Pin_Header_Straight_1x02_Pitch2.54mm" H 6550 16300 50  0001 C CNN
 F 3 "" H 6550 16300 50  0001 C CNN
 	1    6550 16300

Commit message: finish all the tracks
Connections:
- net at U44.5 (Gout): now also U47.1 (Gin); no longer U51.4 (Vin)
- net at U44.6 (Cout): now also U47.2 (Cin); no longer U51.3 (Din)
- net at U44.7 (Dout): now also U47.3 (Din); no longer U51.2 (Cin)
- net at U44.8 (Vout): now also U47.4 (Vin); no longer U51.1 (Gin)
- net at U51.5 (Gout): now also U48.1 (Gin); no longer U47.1 (Gin)
- net at U51.6 (Cout): now also U48.2 (Cin); no longer U47.2 (Cin)
- net at U51.7 (Dout): now also U48.3 (Din); no longer U47.3 (Din)
- net at U51.8 (Vout): now also U48.4 (Vin); no longer U47.4 (Vin)
- net at U47.5 (Gout): now also U51.1 (Gin); no longer U48.1 (Gin)
- net at U47.6 (Cout): now also U51.2 (Cin); no longer U48.2 (Cin)
- net at U47.7 (Dout): now also U51.3 (Din); no longer U48.3 (Din)
- net at U47.8 (Vout): now also U51.4 (Vin); no longer U48.4 (Vin)
