File: sign.sch (KiCad schematic (older format))
At the start: 169 parts, among them J1 CONN_01X02, J10 CONN_01X02, J11 CONN_01X02, J12 CONN_01X02, J13 CONN_01X02, J14 CONN_01X02, J15 CONN_01X02, J16 CONN_01X02, J17 CONN_01X02, J18 CONN_01X02, J19 CONN_01X02, J2 CONN_01X02, J20 CONN_01X02, J21 CONN_01X02, J22 CONN_01X02, J23 CONN_01X02, J24 CONN_01X02, J25 CONN_01X02, J26 CONN_01X02, J27 CONN_01X02, J28 CONN_01X02, J29 CONN_01X02, J3 CONN_01X02, J30 CONN_01X02, J4 CONN_01X02, J5 CONN_01X02, J6 CONN_01X02, J7 CONN_01X02, J8 CONN_01X02, J9 CONN_01X02, U1 APA102C_x6, U10 APA102C_x2, U100 APA102C_x6, U101 APA102C_x4, U102 APA102C_x2, U103 APA102C_x1, U104 APA102C_x3, U105 APA102C_x5, U106 APA102C_x2, U107 APA102C_x3, U108 APA102C_x10, U109 APA102C_x9, U11 APA102C_x2, U110 APA102C_x3, U111 APA102C_x12, U112 APA102C_x16, U113 APA102C_x8, U114 APA102C_x13, U115 APA102C_x3, U116 APA102C_x6, U117 APA102C_x3, U118 APA102C_x6, U119 APA102C_x3, U12 APA102C_x2, U120 APA102C_x2, U121 APA102C_x6, U122 APA102C_x3, U123 APA102C_x6, U124 APA102C_x7, U125 APA102C_x12, U126 APA102C_x6, U127 APA102C_x11, U128 APA102C_x4, U129 APA102C_x6, U13 APA102C_x2, U130 APA102C_x2, U131 APA102C_x2, U132 APA102C_x3, U133 APA102C_x1, U134 APA102C_x3, U135 APA102C_x3, U136 APA102C_x12, U137 APA102C_x12, U138 APA102C_x9, U139 APA102C_x4, U14 APA102C_x3, U15 APA102C_x3, U16 APA102C_x3, U17 APA102C_x3, U18 APA102C_x5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

Commit message: Layout done!
Parts:
- J1, J10, J13, J15, J17, J21, J23, J25, J4, J7: footprint Pin_Headers:Pin_Header_Straight_1x02_Pitch2.54mm -> connector:Power_Connector
- J11, J12, J14, J16, J18, J19, J2, J20, J22, J24, J26, J27, J28, J29, J3, J30, J5, J6, J8, J9: footprint Pin_Headers:Pin_Header_Straight_1x02_Pitch2.54mm -> connector:Sign_Connector
Changed lines of the file:
@@
 F 0 "J1" H 1400 7200 50  0000 C CNN
 F 1 "CONN_01X02" V 1500 7050 50  0000 C CNN
-F 2 "Pin_Headers:Pin_Header_Straight_1x02_Pitch2.54mm" H 1400 7050 50  0001 C CNN
+F 2 "connector:Power_Connector" H 1400 7050 50  0001 C CNN
 F 3 "" H 1400 7050 50  0001 C CNN
 	1    1400 7050
@@
 F 0 "J2" H 1400 7550 50  0000 C CNN
 F 1 "CONN_01X02" V 1500 7400 50  0000 C CNN
-F 2 "Pin_Headers:Pin_Header_Straight_1x02_Pitch2.54mm" H 1400 7400 50  0001 C CNN
+F 2 "connector:Sign_Connector" H 1400 7400 50  0001 C CNN
 F 3 "" H 1400 7400 50  0001 C CNN
 	1    1400 7400
@@
 F 0 "J3" H 1400 7900 50  0000 C CNN
 F 1 "CONN_01X02" V 1500 7750 50  0000 C CNN
-F 2 "Pin_Headers:Pin_Header_Straight_1x02_Pitch2.54mm" H 1400 7750 50  0001 C CNN
+F 2 "connector:Sign_Connector" H 1400 7750 50  0001 C CNN
 F 3 "" H 1400 7750 50  0001 C CNN
 	1    1400 7750
@@
 F 0 "J4" H 8450 7900 50  0000 C CNN
 F 1 "CONN_01X02" V 8550 7750 50  0000 C CNN
-F 2 "Pin_Headers:Pin_Header_Straight_1x02_Pitch2.54mm" H 8450 7750 50  0001 C CNN
+F 2 "connector:Power_Connector" H 8450 7750 50  0001 C CNN
 F 3 "" H 8450 7750 50  0001 C CNN
 	1    8450 7750
@@
 F 0 "J5" H 8450 8250 50  0000 C CNN
 F 1 "CONN_01X02" V 8550 8100 50  0000 C CNN
-F 2 "Pin_Headers:Pin_Header_Straight_1x02_Pitch2.54mm" H 8450 8100 50  0001 C CNN
+F 2 "connector:Sign_Connector" H 8450 8100 50  0001 C CNN
 F 3 "" H 8450 8100 50  0001 C CNN
 	1    8450 8100
@@
 F 0 "J6" H 8450 8600 50  0000 C CNN
 F 1 "CONN_01X02" V 8550 8450 50  0000 C CNN
-F 2 "Pin_Headers:Pin_Header_Straight_1x02_Pitch2.54mm" H 8450 8450 50  0001 C CNN
+F 2 "connector:Sign_Connector" H 8450 8450 50  0001 C CNN
 F 3 "" H 8450 8450 50  0001 C CNN
 	1    8450 8450
@@
 F 0 "J7" H 16250 7900 50  0000 C CNN
 F 1 "CONN_01X02" V 16350 7750 50  0000 C CNN
-F 2 "Pin_Headers:Pin_Header_Straight_1x02_Pitch2.54mm" H 16250 7750 50  0001 C CNN
+F 2 "connector:Power_Connector" H 16250 7750 50  0001 C CNN
 F 3 "" H 16250 7750 50  0001 C CNN
 	1    16250 7750
@@
 F 0 "J8" H 16250 8250 50  0000 C CNN
 F 1 "CONN_01X02" V 16350 8100 50  0000 C CNN
-F 2 "Pin_Headers:Pin_Header_Straight_1x02_Pitch2.54mm" H 16250 8100 50  0001 C CNN
+F 2 "connector:Sign_Connector" H 16250 8100 50  0001 C CNN
 F 3 "" H 16250 8100 50  0001 C CNN
 	1    16250 8100
@@
 F 0 "J9" H 16250 8600 50  0000 C CNN
 F 1 "CONN_01X02" V 16350 8450 50  0000 C CNN
-F 2 "Pin_Headers:Pin_Header_Straight_1x02_Pitch2.54mm" H 16250 8450 50  0001 C CNN
+F 2 "connector:Sign_Connector" H 16250 8450 50  0001 C CNN
 F 3 "" H 16250 8450 50  0001 C CNN
 	1    16250 8450
@@
 F 0 "J23" H 22250 12800 50  0000 C CNN
 F 1 "CONN_01X02" V 22350 12650 50  0000 C CNN
-F 2 "Pin_Headers:Pin_Header_Straight_1x02_Pitch2.54mm" H 22250 12650 50  0001 C CNN
+F 2 "connector:Power_Connector" H 22250 12650 50  0001 C CNN
 F 3 "" H 22250 12650 50  0001 C CNN
 	1    22250 12650
@@
 F 0 "J24" H 22250 13150 50  0000 C CNN
 F 1 "CONN_01X02" V 22350 13000 50  0000 C CNN
-F 2 "Pin_Headers:Pin_Header_Straight_1x02_Pitch2.54mm" H 22250 13000 50  0001 C CNN
+F 2 "connector:Sign_Connector" H 22250 13000 50  0001 C CNN
 F 3 "" H 22250 13000 50  0001 C CNN
 	1    22250 13000
@@
 F 0 "J29" H 24700 4450 50  0000 C CNN
 F 1 "CONN_01X02" V 24800 4300 50  0000 C CNN
-F 2 "Pin_Headers:Pin_Header_Straight_1x02_Pitch2.54mm" H 24700 4300 50  0001 C CNN
+F 2 "connector:Sign_Connector" H 24700 4300 50  0001 C CNN
 F 3 "" H 24700 4300 50  0001 C CNN
 	1    24700 4300
@@
 F 0 "J15" H 16850 16900 50  0000 C CNN
 F 1 "CONN_01X02" V 16950 16750 50  0000 C CNN
-F 2 "Pin_Headers:Pin_Header_Straight_1x02_Pitch2.54mm" H 16850 16750 50  0001 C CNN
+F 2 "connector:Power_Connector" H 16850 16750 50  0001 C CNN
 F 3 "" H 16850 16750 50  0001 C CNN
 	1    16850 16750
@@
 F 0 "J16" H 16850 17250 50  0000 C CNN
 F 1 "CONN_01X02" V 16950 17100 50  0000 C CNN
-F 2 "Pin_Headers:Pin_Header_Straight_1x02_Pitch2.54mm" H 16850 17100 50  0001 C CNN
+F 2 "connector:Sign_Connector" H 16850 17100 50  0001 C CNN
 F 3 "" H 16850 17100 50  0001 C CNN
 	1    16850 17100
@@
 F 0 "J20" H 19350 16550 50  0000 C CNN
 F 1 "CONN_01X02" V 19450 16400 50  0000 C CNN
-F 2 "Pin_Headers:Pin_Header_Straight_1x02_Pitch2.54mm" H 19350 16400 50  0001 C CNN
+F 2 "connector:Sign_Connector" H 19350 16400 50  0001 C CNN
 F 3 "" H 19350 16400 50  0001 C CNN
 	1    19350 16400
@@
 F 0 "J21" H 21050 16900 50  0000 C CNN
 F 1 "CONN_01X02" V 21150 16750 50  0000 C CNN
-F 2 "Pin_Headers:Pin_Header_Straight_1x02_Pitch2.54mm" H 21050 16750 50  0001 C CNN
+F 2 "connector:Power_Connector" H 21050 16750 50  0001 C CNN
 F 3 "" H 21050 16750 50  0001 C CNN
 	1    21050 16750
@@
 F 0 "J22" H 21050 17250 50  0000 C CNN
 F 1 "CONN_01X02" V 21150 17100 50  0000 C CNN
-F 2 "Pin_Headers:Pin_Header_Straight_1x02_Pitch2.54mm" H 21050 17100 50  0001 C CNN
+F 2 "connector:Sign_Connector" H 21050 17100 50  0001 C CNN
 F 3 "" H 21050 17100 50  0001 C CNN
 	1    21050 17100
@@
 F 0 "J28" H 23550 16550 50  0000 C CNN
 F 1 "CONN_01X02" V 23650 16400 50  0000 C CNN
-F 2 "Pin_Headers:Pin_Header_Straight_1x02_Pitch2.54mm" H 23550 16400 50  0001 C CNN
+F 2 "connector:Sign_Connector" H 23550 16400 50  0001 C CNN
 F 3 "" H 23550 16400 50  0001 C CNN
 	1    23550 16400
@@
 F 0 "J13" H 12050 27200 50  0000 C CNN
 F 1 "CONN_01X02" V 12150 27050 50  0000 C CNN
-F 2 "Pin_Headers:Pin_Header_Straight_1x02_Pitch2.54mm" H 12050 27050 50  0001 C CNN
+F 2 "connector:Power_Connector" H 12050 27050 50  0001 C CNN
 F 3 "" H 12050 27050 50  0001 C CNN
 	1    12050 27050
@@
 F 0 "J14" H 12050 27550 50  0000 C CNN
 F 1 "CONN_01X02" V 12150 27400 50  0000 C CNN
-F 2 "Pin_Headers:Pin_Header_Straight_1x02_Pitch2.54mm" H 12050 27400 50  0001 C CNN
+F 2 "connector:Sign_Connector" H 12050 27400 50  0001 C CNN
 F 3 "" H 12050 27400 50  0001 C CNN
 	1    12050 27400
@@
 F 0 "J25" H 22850 25300 50  0000 C CNN
 F 1 "CONN_01X02" V 22950 25150 50  0000 C CNN
-F 2 "Pin_Headers:Pin_Header_Straight_1x02_Pitch2.54mm" H 22850 25150 50  0001 C CNN
+F 2 "connector:Power_Connector" H 22850 25150 50  0001 C CNN
 F 3 "" H 22850 25150 50  0001 C CNN
 	1    22850 25150
@@
 F 0 "J26" H 22850 25650 50  0000 C CNN
 F 1 "CONN_01X02" V 22950 25500 50  0000 C CNN
-F 2 "Pin_Headers:Pin_Header_Straight_1x02_Pitch2.54mm" H 22850 25500 50  0001 C CNN
+F 2 "connector:Sign_Connector" H 22850 25500 50  0001 C CNN
 F 3 "" H 22850 25500 50  0001 C CNN
 	1    22850 25500
@@
 F 0 "J17" H 18650 25350 50  0000 C CNN
 F 1 "CONN_01X02" V 18750 25200 50  0000 C CNN
-F 2 "Pin_Headers:Pin_Header_Straight_1x02_Pitch2.54mm" H 18650 25200 50  0001 C CNN
+F 2 "connector:Power_Connector" H 18650 25200 50  0001 C CNN
 F 3 "" H 18650 25200 50  0001 C CNN
 	1    18650 25200
@@
 F 0 "J18" H 18650 25700 50  0000 C CNN
 F 1 "CONN_01X02" V 18750 25550 50  0000 C CNN
-F 2 "Pin_Headers:Pin_Header_Straight_1x02_Pitch2.54mm" H 18650 25550 50  0001 C CNN
+F 2 "connector:Sign_Connector" H 18650 25550 50  0001 C CNN
 F 3 "" H 18650 25550 50  0001 C CNN
 	1    18650 25550
@@
 F 0 "J10" H 5450 17400 50  0000 C CNN
 F 1 "CONN_01X02" V 5550 17250 50  0000 C CNN
-F 2 "Pin_Headers:Pin_Header_Straight_1x02_Pitch2.54mm" H 5450 17250 50  0001 C CNN
+F 2 "connector:Power_Connector" H 5450 17250 50  0001 C CNN
 F 3 "" H 5450 17250 50  0001 C CNN
 	1    5450 17250
@@
 F 0 "J11" H 5450 17750 50  0000 C CNN
 F 1 "CONN_01X02" V 5550 17600 50  0000 C CNN
-F 2 "Pin_Headers:Pin_Header_Straight_1x02_Pitch2.54mm" H 5450 17600 50  0001 C CNN
+F 2 "connector:Sign_Connector" H 5450 17600 50  0001 C CNN
 F 3 "" H 5450 17600 50  0001 C CNN
 	1    5450 17600
@@
 F 0 "J19" H 18900 19050 50  0000 C CNN
 F 1 "CONN_01X02" V 19000 18900 50  0000 C CNN
-F 2 "Pin_Headers:Pin_Header_Straight_1x02_Pitch2.54mm" H 18900 18900 50  0001 C CNN
+F 2 "connector:Sign_Connector" H 18900 18900 50  0001 C CNN
 F 3 "" H 18900 18900 50  0001 C CNN
 	1    18900 18900
@@
 F 0 "J27" H 23100 19100 50  0000 C CNN
 F 1 "CONN_01X02" V 23200 18950 50  0000 C CNN
-F 2 "Pin_Headers:Pin_Header_Straight_1x02_Pitch2.54mm" H 23100 18950 50  0001 C CNN
+F 2 "connector:Sign_Connector" H 23100 18950 50  0001 C CNN
 F 3 "" H 23100 18950 50  0001 C CNN
 	1    23100 18950
@@
 F 0 "J30" H 34500 23300 50  0000 C CNN
 F 1 "CONN_01X02" V 34600 23150 50  0000 C CNN
-F 2 "Pin_Headers:Pin_Header_Straight_1x02_Pitch2.54mm" H 34500 23150 50  0001 C CNN
+F 2 "connector:Sign_Connector" H 34500 23150 50  0001 C CNN
 F 3 "" H 34500 23150 50  0001 C CNN
 	1    34500 23150
@@
 F 0 "J12" H 6550 16450 50  0000 C CNN
 F 1 "CONN_01X02" V 6650 16300 50  0000 C CNN
-F 2 "Pin_Headers:Pin_Header_Straight_1x02_Pitch2.54mm" H 6550 16300 50  0001 C CNN
+F 2 "connector:Sign_Connector" H 6550 16300 50  0001 C CNN
 F 3 "" H 6550 16300 50  0001 C CNN
 	1    6550 16300
