File: sign.kicad_pcb (KiCad board)
At the start: 2 copper layers, 767.9 x 642.9 mm, 142 parts, among them J1 CONN_01X02, J2 CONN_01X02, J3 CONN_01X02, U1 APA102C_x6, U10 APA102C_x2, U100 APA102C_x6, U101 APA102C_x4, U102 APA102C_x2, U103 APA102C_x1, U104 APA102C_x3, U105 APA102C_x5, U106 APA102C_x2, U107 APA102C_x3, U108 APA102C_x10, U109 APA102C_x9, U11 APA102C_x2, U110 APA102C_x3, U111 APA102C_x12, U112 APA102C_x16, U113 APA102C_x8, U114 APA102C_x13, U115 APA102C_x3, U116 APA102C_x6, U117 APA102C_x3, U118 APA102C_x6, U119 APA102C_x3, U12 APA102C_x2, U120 APA102C_x2, U121 APA102C_x6, U122 APA102C_x3, U123 APA102C_x6, U124 APA102C_x7, U125 APA102C_x12, U126 APA102C_x6, U127 APA102C_x11, U128 APA102C_x4, U129 APA102C_x6, U13 APA102C_x2, U130 APA102C_x2, U131 APA102C_x2, U132 APA102C_x3, U133 APA102C_x1, U134 APA102C_x3, U135 APA102C_x3, U136 APA102C_x12, U137 APA102C_x12, U138 APA102C_x9, U139 APA102C_x4, U14 APA102C_x3, U15 APA102C_x3, U16 APA102C_x3, U17 APA102C_x3, U18 APA102C_x5, U19 APA102C_x6, U2 APA102C_x8, U20 APA102C_x2, U21 APA102C_x7, U22 APA102C_x5, U23 APA102C_x7, U24 APA102C_x3, U25 APA102C_x2, U26 APA102C_x7, U27 APA102C_x2, U28 APA102C_x3, U29 APA102C_x5, U3 APA102C_x11, U30 APA102C_x2, U31 APA102C_x5, U32 APA102C_x2, U33 APA102C_x8, U34 APA102C_x9, U35 APA102C_x3, U36 APA102C_x2, U37 APA102C_x5, U38 APA102C_x11, U39 APA102C_x6, U4 APA102C_x6, U40 APA102C_x4, U41 APA102C_x5, U42 APA102C_x3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

Commit message: Untangle all the pcb letters and wire up both d's.
Parts:
- added J10: CONN_01X02, Pin_Headers:Pin_Header_Straight_1x02_Pitch2.54mm, F.Cu at (481.8, 330.5)
- added J11: CONN_01X02, Pin_Headers:Pin_Header_Straight_1x02_Pitch2.54mm, F.Cu at (118.4, 403.6)
- added J12: CONN_01X02, Pin_Headers:Pin_Header_Straight_1x02_Pitch2.54mm, F.Cu at (140.0, 350.0)
- added J13: CONN_01X02, Pin_Headers:Pin_Header_Straight_1x02_Pitch2.54mm, F.Cu at (199.4, 276.9)
- added J14: CONN_01X02, Pin_Headers:Pin_Header_Straight_1x02_Pitch2.54mm, F.Cu at (230.1, 618.2)
- added J15: CONN_01X02, Pin_Headers:Pin_Header_Straight_1x02_Pitch2.54mm, F.Cu at (29.5, 114.0)
- added J16: CONN_01X02, Pin_Headers:Pin_Header_Straight_1x02_Pitch2.54mm, F.Cu at (380.5, 397.5)
- added J17: CONN_01X02, Pin_Headers:Pin_Header_Straight_1x02_Pitch2.54mm, F.Cu at (373.1, 279.1)
- added J18: CONN_01X02, Pin_Headers:Pin_Header_Straight_1x02_Pitch2.54mm, F.Cu at (474.5, 617.7)
- added J19: CONN_01X02, Pin_Headers:Pin_Header_Straight_1x02_Pitch2.54mm, F.Cu at (451.1, 433.6)
- added J20: CONN_01X02, Pin_Headers:Pin_Header_Straight_1x02_Pitch2.54mm, F.Cu at (462.3, 361.9)
- added J21: CONN_01X02, Pin_Headers:Pin_Header_Straight_1x02_Pitch2.54mm, F.Cu at (589.5, 634.2)
- added J22: CONN_01X02, Pin_Headers:Pin_Header_Straight_1x02_Pitch2.54mm, F.Cu at (484.6, 405.6)
- added J23: CONN_01X02, Pin_Headers:Pin_Header_Straight_1x02_Pitch2.54mm, F.Cu at (487.4, 301.2)
- added J24: CONN_01X02, Pin_Headers:Pin_Header_Straight_1x02_Pitch2.54mm, F.Cu at (521.2, 339.9)
- added J25: CONN_01X02, Pin_Headers:Pin_Header_Straight_1x02_Pitch2.54mm, F.Cu at (440.4, 621.3)
- added J26: CONN_01X02, Pin_Headers:Pin_Header_Straight_1x02_Pitch2.54mm, F.Cu at (541.3, 621.8)
- added J27: CONN_01X02, Pin_Headers:Pin_Header_Straight_1x02_Pitch2.54mm, F.Cu at (544.8, 422.7)
- added J28: CONN_01X02, Pin_Headers:Pin_Header_Straight_1x02_Pitch2.54mm, F.Cu at (565.9, 366.5)
- added J29: CONN_01X02, Pin_Headers:Pin_Header_Straight_1x02_Pitch2.54mm, F.Cu at (603.8, 75.9)
- added J30: CONN_01X02, Pin_Headers:Pin_Header_Straight_1x02_Pitch2.54mm, F.Cu at (837.4, 447.3)
- added J4: CONN_01X02, Pin_Headers:Pin_Header_Straight_1x02_Pitch2.54mm, F.Cu at (515.6, 311.7)
- added J5: CONN_01X02, Pin_Headers:Pin_Header_Straight_1x02_Pitch2.54mm, F.Cu at (214.4, 276.9)
- added J6: CONN_01X02, Pin_Headers:Pin_Header_Straight_1x02_Pitch2.54mm, F.Cu at (378.5, 676.1)
- added J7: CONN_01X02, Pin_Headers:Pin_Header_Straight_1x02_Pitch2.54mm, F.Cu at (285.0, 402.8)
- added J8: CONN_01X02, Pin_Headers:Pin_Header_Straight_1x02_Pitch2.54mm, F.Cu at (404.6, 279.7)
- added J9: CONN_01X02, Pin_Headers:Pin_Header_Straight_1x02_Pitch2.54mm, F.Cu at (439.9, 78.2)
- J1, J2, J3: footprint Pin_Headers:Pin_Header_Straight_1x02 -> Pin_Headers:Pin_Header_Straight_1x02_Pitch2.54mm
- moved J1 550.2 mm to (287.8, 672.3), turned to 0 degrees
- moved J3 98.4 mm to (117.3, 154.9), turned to 0 degrees
- moved J2 40.9 mm to (30.2, 165.6), turned to 0 degrees
- turned U100 to 270 degrees
- turned U102 to 270 degrees
- turned U104 to 270 degrees
- turned U106 to 270 degrees
- turned U108 to 270 degrees
- turned U110 to 270 degrees
- turned U113 to 270 degrees
- turned U114 to 270 degrees
- turned U117 to 270 degrees
- turned U118 to 270 degrees
- turned U122 to 270 degrees
- turned U123 to 270 degrees
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Connections:
- U101 pad 1: (no net) -> Net-(U101-Pad1)
- U101 pad 2: (no net) -> Net-(U101-Pad2)
- U101 pad 3: (no net) -> Net-(U101-Pad3)
- U101 pad 4: (no net) -> Net-(U101-Pad4)
- U101 pad 5: (no net) -> Net-(U101-Pad5)
- U101 pad 6: (no net) -> Net-(U101-Pad6)
- U101 pad 7: (no net) -> Net-(U101-Pad7)
- U101 pad 8: (no net) -> Net-(U101-Pad8)
- U102 pad 1: (no net) -> GND
- U102 pad 2: (no net) -> Net-(J26-Pad1)
- U102 pad 3: (no net) -> Net-(J26-Pad2)
- U102 pad 4: (no net) -> +5V
- U102 pad 5: (no net) -> Net-(U102-Pad5)
- U102 pad 6: (no net) -> Net-(U102-Pad6)
- U102 pad 7: (no net) -> Net-(U102-Pad7)
- U102 pad 8: (no net) -> Net-(U102-Pad8)
- U104 pad 1: (no net) -> Net-(U101-Pad5)
- U104 pad 2: (no net) -> Net-(U101-Pad6)
- U104 pad 3: (no net) -> Net-(U101-Pad7)
- U104 pad 4: (no net) -> Net-(U101-Pad8)
- U104 pad 5: (no net) -> Net-(U104-Pad5)
- U104 pad 6: (no net) -> Net-(U104-Pad6)
- U104 pad 7: (no net) -> Net-(U104-Pad7)
- U104 pad 8: (no net) -> Net-(U104-Pad8)
- U105 pad 1: (no net) -> Net-(U102-Pad5)
- U105 pad 2: (no net) -> Net-(U102-Pad6)
- U105 pad 3: (no net) -> Net-(U102-Pad7)
- U105 pad 4: (no net) -> Net-(U102-Pad8)
- U105 pad 5: (no net) -> Net-(U105-Pad5)
- U105 pad 6: (no net) -> Net-(U105-Pad6)
- U105 pad 7: (no net) -> Net-(U105-Pad7)
- U105 pad 8: (no net) -> Net-(U105-Pad8)
- U106 pad 1: (no net) -> Net-(U106-Pad1)
- U106 pad 2: (no net) -> Net-(U106-Pad2)
- U106 pad 3: (no net) -> Net-(U106-Pad3)
- U106 pad 4: (no net) -> Net-(U106-Pad4)
- U106 pad 6: (no net) -> Net-(J29-Pad1)
- U106 pad 7: (no net) -> Net-(J29-Pad2)
- U107 pad 1: (no net) -> Net-(U104-Pad5)
- U107 pad 2: (no net) -> Net-(U104-Pad6)
- U107 pad 3: (no net) -> Net-(U104-Pad7)
- U107 pad 4: (no net) -> Net-(U104-Pad8)
- U107 pad 5: (no net) -> Net-(U107-Pad5)
- U107 pad 6: (no net) -> Net-(U107-Pad6)
- U107 pad 7: (no net) -> Net-(U107-Pad7)
- U107 pad 8: (no net) -> Net-(U107-Pad8)
- U108 pad 1: (no net) -> Net-(U105-Pad5)
- U108 pad 2: (no net) -> Net-(U105-Pad6)
- U108 pad 3: (no net) -> Net-(U105-Pad7)
- U108 pad 4: (no net) -> Net-(U105-Pad8)
- U108 pad 5: (no net) -> Net-(U108-Pad5)
- U108 pad 6: (no net) -> Net-(U108-Pad6)
- U108 pad 7: (no net) -> Net-(U108-Pad7)
- U108 pad 8: (no net) -> Net-(U108-Pad8)
- U109 pad 1: (no net) -> Net-(U109-Pad1)
- U109 pad 2: (no net) -> Net-(U109-Pad2)
- U109 pad 3: (no net) -> Net-(U109-Pad3)
- U109 pad 4: (no net) -> Net-(U109-Pad4)
- U109 pad 5: (no net) -> Net-(U106-Pad1)
- U109 pad 6: (no net) -> Net-(U106-Pad2)
- U109 pad 7: (no net) -> Net-(U106-Pad3)
- U109 pad 8: (no net) -> Net-(U106-Pad4)
- U110 pad 1: (no net) -> Net-(U107-Pad5)
- U110 pad 2: (no net) -> Net-(U107-Pad6)
- U110 pad 3: (no net) -> Net-(U107-Pad7)
- U110 pad 4: (no net) -> Net-(U107-Pad8)
- U110 pad 5: (no net) -> Net-(U110-Pad5)
- U110 pad 6: (no net) -> Net-(U110-Pad6)
- U110 pad 7: (no net) -> Net-(U110-Pad7)
- U110 pad 8: (no net) -> Net-(U110-Pad8)
- U111 pad 1: (no net) -> Net-(U108-Pad5)
- U111 pad 2: (no net) -> Net-(U108-Pad6)
- U111 pad 3: (no net) -> Net-(U108-Pad7)
- U111 pad 4: (no net) -> Net-(U108-Pad8)
- U111 pad 5: (no net) -> Net-(U111-Pad5)
- U111 pad 6: (no net) -> Net-(U111-Pad6)
- U111 pad 7: (no net) -> Net-(U111-Pad7)
- U111 pad 8: (no net) -> Net-(U111-Pad8)
- U112 pad 1: (no net) -> Net-(U110-Pad5)
- U112 pad 2: (no net) -> Net-(U110-Pad6)
- U112 pad 3: (no net) -> Net-(U110-Pad7)
- U112 pad 4: (no net) -> Net-(U110-Pad8)
- U112 pad 5: (no net) -> Net-(U112-Pad5)
- U112 pad 6: (no net) -> Net-(U112-Pad6)
- U112 pad 7: (no net) -> Net-(U112-Pad7)
- U112 pad 8: (no net) -> Net-(U112-Pad8)
- U113 pad 1: (no net) -> Net-(U111-Pad5)
- U113 pad 2: (no net) -> Net-(U111-Pad6)
- U113 pad 3: (no net) -> Net-(U111-Pad7)
- U113 pad 4: (no net) -> Net-(U111-Pad8)
- U113 pad 5: (no net) -> Net-(U113-Pad5)
- U113 pad 6: (no net) -> Net-(U113-Pad6)
- U113 pad 7: (no net) -> Net-(U113-Pad7)
- U113 pad 8: (no net) -> Net-(U113-Pad8)
- U114 pad 1: (no net) -> Net-(U112-Pad5)
- U114 pad 2: (no net) -> Net-(U112-Pad6)
- U114 pad 3: (no net) -> Net-(U112-Pad7)
- U114 pad 4: (no net) -> Net-(U112-Pad8)
- U114 pad 5: (no net) -> Net-(U114-Pad5)
- U114 pad 6: (no net) -> Net-(U114-Pad6)
- U114 pad 7: (no net) -> Net-(U114-Pad7)
- U114 pad 8: (no net) -> Net-(U114-Pad8)
- U115 pad 1: (no net) -> Net-(U113-Pad5)
- U115 pad 2: (no net) -> Net-(U113-Pad6)
- U115 pad 3: (no net) -> Net-(U113-Pad7)
- U115 pad 4: (no net) -> Net-(U113-Pad8)
- U115 pad 5: (no net) -> Net-(U115-Pad5)
- U115 pad 6: (no net) -> Net-(U115-Pad6)
- U115 pad 7: (no net) -> Net-(U115-Pad7)
- U115 pad 8: (no net) -> Net-(U115-Pad8)
- U116 pad 1: (no net) -> Net-(U114-Pad5)
- U116 pad 2: (no net) -> Net-(U114-Pad6)
- U116 pad 3: (no net) -> Net-(U114-Pad7)
- U116 pad 4: (no net) -> Net-(U114-Pad8)
- U116 pad 5: (no net) -> Net-(U116-Pad5)
- U116 pad 6: (no net) -> Net-(U116-Pad6)
- U116 pad 7: (no net) -> Net-(U116-Pad7)
- U116 pad 8: (no net) -> Net-(U116-Pad8)
- U117 pad 1: (no net) -> Net-(U115-Pad5)
- U117 pad 2: (no net) -> Net-(U115-Pad6)
- U117 pad 3: (no net) -> Net-(U115-Pad7)
- U117 pad 4: (no net) -> Net-(U115-Pad8)
- U117 pad 5: (no net) -> Net-(U117-Pad5)
- U117 pad 6: (no net) -> Net-(U117-Pad6)
- U117 pad 7: (no net) -> Net-(U117-Pad7)
- U117 pad 8: (no net) -> Net-(U117-Pad8)
- U118 pad 1: (no net) -> Net-(U116-Pad5)
- U118 pad 2: (no net) -> Net-(U116-Pad6)
- U118 pad 3: (no net) -> Net-(U116-Pad7)
- U118 pad 4: (no net) -> Net-(U116-Pad8)
- U118 pad 5: (no net) -> Net-(U118-Pad5)
- U118 pad 6: (no net) -> Net-(U118-Pad6)
- U118 pad 7: (no net) -> Net-(U118-Pad7)
- U118 pad 8: (no net) -> Net-(U118-Pad8)
- U119 pad 1: (no net) -> Net-(U117-Pad5)
- U119 pad 2: (no net) -> Net-(U117-Pad6)
- U119 pad 3: (no net) -> Net-(U117-Pad7)
- U119 pad 4: (no net) -> Net-(U117-Pad8)
- U119 pad 5: (no net) -> Net-(U119-Pad5)
- U119 pad 6: (no net) -> Net-(U119-Pad6)
- U119 pad 7: (no net) -> Net-(U119-Pad7)
- U119 pad 8: (no net) -> Net-(U119-Pad8)
- U120 pad 1: (no net) -> Net-(U120-Pad1)
- U120 pad 2: (no net) -> Net-(U120-Pad2)
- U120 pad 3: (no net) -> Net-(U120-Pad3)
- U120 pad 4: (no net) -> Net-(U120-Pad4)
- U120 pad 5: (no net) -> Net-(U120-Pad5)
- U120 pad 6: (no net) -> Net-(U120-Pad6)
- U120 pad 7: (no net) -> Net-(U120-Pad7)
- U120 pad 8: (no net) -> Net-(U120-Pad8)
- U121 pad 1: (no net) -> Net-(U118-Pad5)
- U121 pad 2: (no net) -> Net-(U118-Pad6)
- U121 pad 3: (no net) -> Net-(U118-Pad7)
- U121 pad 4: (no net) -> Net-(U118-Pad8)
- U121 pad 5: (no net) -> Net-(U121-Pad5)
- U121 pad 6: (no net) -> Net-(U121-Pad6)
- U121 pad 7: (no net) -> Net-(U121-Pad7)
- U121 pad 8: (no net) -> Net-(U121-Pad8)
- U122 pad 1: (no net) -> Net-(U119-Pad5)
- U122 pad 2: (no net) -> Net-(U119-Pad6)
- U122 pad 3: (no net) -> Net-(U119-Pad7)
- U122 pad 4: (no net) -> Net-(U119-Pad8)
- U122 pad 5: (no net) -> Net-(U122-Pad5)
- U122 pad 6: (no net) -> Net-(U122-Pad6)
- U122 pad 7: (no net) -> Net-(U122-Pad7)
- U122 pad 8: (no net) -> Net-(U122-Pad8)
- U123 pad 1: (no net) -> Net-(U122-Pad5)
- U123 pad 2: (no net) -> Net-(U122-Pad6)
- U123 pad 3: (no net) -> Net-(U122-Pad7)
- U123 pad 4: (no net) -> Net-(U122-Pad8)
- U123 pad 5: (no net) -> Net-(U120-Pad1)
- U123 pad 6: (no net) -> Net-(U120-Pad2)
- U123 pad 7: (no net) -> Net-(U120-Pad3)
- U123 pad 8: (no net) -> Net-(U120-Pad4)
- U124 pad 1: (no net) -> Net-(U121-Pad5)
- U124 pad 2: (no net) -> Net-(U121-Pad6)
- U124 pad 3: (no net) -> Net-(U121-Pad7)
- U124 pad 4: (no net) -> Net-(U121-Pad8)
- U124 pad 5: (no net) -> Net-(U124-Pad5)
- U124 pad 6: (no net) -> Net-(U124-Pad6)
- U124 pad 7: (no net) -> Net-(U124-Pad7)
- U124 pad 8: (no net) -> Net-(U124-Pad8)
- U125 pad 1: (no net) -> Net-(U120-Pad5)
- U125 pad 2: (no net) -> Net-(U120-Pad6)
- U125 pad 3: (no net) -> Net-(U120-Pad7)
- U125 pad 4: (no net) -> Net-(U120-Pad8)
- U125 pad 5: (no net) -> Net-(U125-Pad5)
- U125 pad 6: (no net) -> Net-(U125-Pad6)
- U125 pad 7: (no net) -> Net-(U125-Pad7)
- U125 pad 8: (no net) -> Net-(U125-Pad8)
- U126 pad 1: (no net) -> Net-(U124-Pad5)
- U126 pad 2: (no net) -> Net-(U124-Pad6)
- U126 pad 3: (no net) -> Net-(U124-Pad7)
- U126 pad 4: (no net) -> Net-(U124-Pad8)
- U126 pad 5: (no net) -> Net-(U126-Pad5)
- U126 pad 6: (no net) -> Net-(U126-Pad6)
- U126 pad 7: (no net) -> Net-(U126-Pad7)
- U126 pad 8: (no net) -> Net-(U126-Pad8)
- U127 pad 1: (no net) -> Net-(U125-Pad5)
- U127 pad 2: (no net) -> Net-(U125-Pad6)
- U127 pad 3: (no net) -> Net-(U125-Pad7)
- U127 pad 4: (no net) -> Net-(U125-Pad8)
- U127 pad 5: (no net) -> Net-(U127-Pad5)
- U127 pad 6: (no net) -> Net-(U127-Pad6)
- U127 pad 7: (no net) -> Net-(U127-Pad7)
- U127 pad 8: (no net) -> Net-(U127-Pad8)
- U128 pad 1: (no net) -> Net-(U126-Pad5)
- U128 pad 2: (no net) -> Net-(U126-Pad6)
- U128 pad 3: (no net) -> Net-(U126-Pad7)
- U128 pad 4: (no net) -> Net-(U126-Pad8)
- U128 pad 5: (no net) -> Net-(U128-Pad5)
- U128 pad 6: (no net) -> Net-(U128-Pad6)
- U128 pad 7: (no net) -> Net-(U128-Pad7)
- U128 pad 8: (no net) -> Net-(U128-Pad8)
- U129 pad 1: (no net) -> Net-(U127-Pad5)
- U129 pad 2: (no net) -> Net-(U127-Pad6)
- U129 pad 3: (no net) -> Net-(U127-Pad7)
- U129 pad 4: (no net) -> Net-(U127-Pad8)
- U129 pad 5: (no net) -> Net-(U129-Pad5)
- U129 pad 6: (no net) -> Net-(U129-Pad6)
- U129 pad 7: (no net) -> Net-(U129-Pad7)
- U129 pad 8: (no net) -> Net-(U129-Pad8)
- U130 pad 1: (no net) -> Net-(U128-Pad5)
- U130 pad 2: (no net) -> Net-(U128-Pad6)
- U130 pad 3: (no net) -> Net-(U128-Pad7)
- U130 pad 4: (no net) -> Net-(U128-Pad8)
- U130 pad 5: (no net) -> Net-(U109-Pad1)
- U130 pad 6: (no net) -> Net-(U109-Pad2)
- U130 pad 7: (no net) -> Net-(U109-Pad3)
- U130 pad 8: (no net) -> Net-(U109-Pad4)
- U131 pad 1: (no net) -> Net-(U129-Pad5)
- U131 pad 2: (no net) -> Net-(U129-Pad6)
- U131 pad 3: (no net) -> Net-(U129-Pad7)
- U131 pad 4: (no net) -> Net-(U129-Pad8)
- U131 pad 5: (no net) -> Net-(U131-Pad5)
- U131 pad 6: (no net) -> Net-(U131-Pad6)
- U131 pad 7: (no net) -> Net-(U131-Pad7)
- U131 pad 8: (no net) -> Net-(U131-Pad8)
- U132 pad 1: (no net) -> Net-(U131-Pad5)
- U132 pad 2: (no net) -> Net-(U131-Pad6)
- U132 pad 3: (no net) -> Net-(U131-Pad7)
- U132 pad 4: (no net) -> Net-(U131-Pad8)
- U132 pad 5: (no net) -> Net-(U132-Pad5)
- U132 pad 6: (no net) -> Net-(U132-Pad6)
- U132 pad 7: (no net) -> Net-(U132-Pad7)
- U132 pad 8: (no net) -> Net-(U132-Pad8)
- U133 pad 1: (no net) -> Net-(U133-Pad1)
- U133 pad 2: (no net) -> Net-(U133-Pad2)
- U133 pad 3: (no net) -> Net-(U133-Pad3)
- U133 pad 4: (no net) -> Net-(U133-Pad4)
- U133 pad 5: (no net) -> Net-(U133-Pad5)
- U133 pad 6: (no net) -> Net-(U133-Pad6)
- U133 pad 7: (no net) -> Net-(U133-Pad7)
- U133 pad 8: (no net) -> Net-(U133-Pad8)
- U134 pad 1: (no net) -> Net-(U132-Pad5)
- U134 pad 2: (no net) -> Net-(U132-Pad6)
- U134 pad 3: (no net) -> Net-(U132-Pad7)
- U134 pad 4: (no net) -> Net-(U132-Pad8)
- U134 pad 5: (no net) -> Net-(U134-Pad5)
- U134 pad 6: (no net) -> Net-(U134-Pad6)
- U134 pad 7: (no net) -> Net-(U134-Pad7)
- U134 pad 8: (no net) -> Net-(U134-Pad8)
- U135 pad 1: (no net) -> Net-(U134-Pad5)
- U135 pad 2: (no net) -> Net-(U134-Pad6)
- U135 pad 3: (no net) -> Net-(U134-Pad7)
- U135 pad 4: (no net) -> Net-(U134-Pad8)
- U135 pad 5: (no net) -> Net-(U133-Pad1)
- U135 pad 6: (no net) -> Net-(U133-Pad2)
- U135 pad 7: (no net) -> Net-(U133-Pad3)
- U135 pad 8: (no net) -> Net-(U133-Pad4)
- U136 pad 1: (no net) -> Net-(U133-Pad5)
- U136 pad 2: (no net) -> Net-(U133-Pad6)
- U136 pad 3: (no net) -> Net-(U133-Pad7)
- U136 pad 4: (no net) -> Net-(U133-Pad8)
- U136 pad 5: (no net) -> Net-(U136-Pad5)
- U136 pad 6: (no net) -> Net-(U136-Pad6)
- U136 pad 7: (no net) -> Net-(U136-Pad7)
- U136 pad 8: (no net) -> Net-(U136-Pad8)
- U137 pad 1: (no net) -> Net-(U136-Pad5)
- U137 pad 2: (no net) -> Net-(U136-Pad6)
- U137 pad 3: (no net) -> Net-(U136-Pad7)
- U137 pad 4: (no net) -> Net-(U136-Pad8)
- U137 pad 5: (no net) -> Net-(U137-Pad5)
- U137 pad 6: (no net) -> Net-(U137-Pad6)
- U137 pad 7: (no net) -> Net-(U137-Pad7)
- U137 pad 8: (no net) -> Net-(U137-Pad8)
- U138 pad 1: (no net) -> Net-(U137-Pad5)
- U138 pad 2: (no net) -> Net-(U137-Pad6)
- U138 pad 3: (no net) -> Net-(U137-Pad7)
- U138 pad 4: (no net) -> Net-(U137-Pad8)
- U138 pad 5: (no net) -> Net-(U138-Pad5)
- U138 pad 6: (no net) -> Net-(U138-Pad6)
- U138 pad 7: (no net) -> Net-(U138-Pad7)
- U138 pad 8: (no net) -> Net-(U138-Pad8)
- U139 pad 1: (no net) -> Net-(U138-Pad5)
- U139 pad 2: (no net) -> Net-(U138-Pad6)
- U139 pad 3: (no net) -> Net-(U138-Pad7)
- U139 pad 4: (no net) -> Net-(U138-Pad8)
- U139 pad 6: (no net) -> Net-(J30-Pad1)
- U139 pad 7: (no net) -> Net-(J30-Pad2)
- U18 pad 1: (no net) -> Net-(U18-Pad1)
- U18 pad 2: (no net) -> Net-(U18-Pad2)
- U18 pad 3: (no net) -> Net-(U18-Pad3)
- U18 pad 4: (no net) -> Net-(U18-Pad4)
- U18 pad 5: (no net) -> Net-(U18-Pad5)
- U18 pad 6: (no net) -> Net-(U18-Pad6)
- U18 pad 7: (no net) -> Net-(U18-Pad7)
- U18 pad 8: (no net) -> Net-(U18-Pad8)
- U21 pad 1: (no net) -> Net-(U21-Pad1)
- U21 pad 2: (no net) -> Net-(U21-Pad2)
- U21 pad 3: (no net) -> Net-(U21-Pad3)
- U21 pad 4: (no net) -> Net-(U21-Pad4)
- U21 pad 5: (no net) -> Net-(U18-Pad1)
- U21 pad 6: (no net) -> Net-(U18-Pad2)
- U21 pad 7: (no net) -> Net-(U18-Pad3)
- U21 pad 8: (no net) -> Net-(U18-Pad4)
- U23 pad 1: (no net) -> Net-(U18-Pad5)
- U23 pad 2: (no net) -> Net-(U18-Pad6)
- U23 pad 3: (no net) -> Net-(U18-Pad7)
- U23 pad 4: (no net) -> Net-(U18-Pad8)
- U23 pad 6: (no net) -> Net-(J12-Pad1)
- U23 pad 7: (no net) -> Net-(J12-Pad2)
- U24 pad 1: (no net) -> Net-(U24-Pad1)
- U24 pad 2: (no net) -> Net-(U24-Pad2)
- U24 pad 3: (no net) -> Net-(U24-Pad3)
- U24 pad 4: (no net) -> Net-(U24-Pad4)
- U24 pad 5: (no net) -> Net-(U21-Pad1)
- U24 pad 6: (no net) -> Net-(U21-Pad2)
- U24 pad 7: (no net) -> Net-(U21-Pad3)
- U24 pad 8: (no net) -> Net-(U21-Pad4)
- U26 pad 1: (no net) -> Net-(U26-Pad1)
- U26 pad 2: (no net) -> Net-(U26-Pad2)
- U26 pad 3: (no net) -> Net-(U26-Pad3)
- U26 pad 4: (no net) -> Net-(U26-Pad4)
- U26 pad 5: (no net) -> Net-(U26-Pad5)
- U26 pad 6: (no net) -> Net-(U26-Pad6)
- U26 pad 7: (no net) -> Net-(U26-Pad7)
- U26 pad 8: (no net) -> Net-(U26-Pad8)
- U27 pad 1: (no net) -> Net-(U27-Pad1)
- U27 pad 2: (no net) -> Net-(U27-Pad2)
- U27 pad 3: (no net) -> Net-(U27-Pad3)
- U27 pad 4: (no net) -> Net-(U27-Pad4)
- U27 pad 5: (no net) -> Net-(U24-Pad1)
- U27 pad 6: (no net) -> Net-(U24-Pad2)
- U27 pad 7: (no net) -> Net-(U24-Pad3)
- U27 pad 8: (no net) -> Net-(U24-Pad4)
- U28 pad 1: (no net) -> Net-(U28-Pad1)
- U28 pad 2: (no net) -> Net-(U28-Pad2)
- U28 pad 3: (no net) -> Net-(U28-Pad3)
- U28 pad 4: (no net) -> Net-(U28-Pad4)
- U28 pad 5: (no net) -> Net-(U26-Pad1)
- U28 pad 6: (no net) -> Net-(U26-Pad2)
- U28 pad 7: (no net) -> Net-(U26-Pad3)
- U28 pad 8: (no net) -> Net-(U26-Pad4)
- U29 pad 1: (no net) -> Net-(U26-Pad5)
- U29 pad 2: (no net) -> Net-(U26-Pad6)
- U29 pad 3: (no net) -> Net-(U26-Pad7)
- U29 pad 4: (no net) -> Net-(U26-Pad8)
- U29 pad 5: (no net) -> Net-(U29-Pad5)
- U29 pad 6: (no net) -> Net-(U29-Pad6)
- U29 pad 7: (no net) -> Net-(U29-Pad7)
- U29 pad 8: (no net) -> Net-(U29-Pad8)
- U30 pad 1: (no net) -> Net-(U30-Pad1)
- U30 pad 2: (no net) -> Net-(U30-Pad2)
- U30 pad 3: (no net) -> Net-(U30-Pad3)
- U30 pad 4: (no net) -> Net-(U30-Pad4)
- U30 pad 5: (no net) -> Net-(U27-Pad1)
- U30 pad 6: (no net) -> Net-(U27-Pad2)
- U30 pad 7: (no net) -> Net-(U27-Pad3)
- U30 pad 8: (no net) -> Net-(U27-Pad4)
- U31 pad 2: (no net) -> Net-(J5-Pad1)
- U31 pad 3: (no net) -> Net-(J5-Pad2)
- U32 pad 1: (no net) -> Net-(U32-Pad1)
- U32 pad 2: (no net) -> Net-(U32-Pad2)
- U32 pad 3: (no net) -> Net-(U32-Pad3)
- U32 pad 4: (no net) -> Net-(U32-Pad4)
- U32 pad 5: (no net) -> Net-(U28-Pad1)
- U32 pad 6: (no net) -> Net-(U28-Pad2)
- U32 pad 7: (no net) -> Net-(U28-Pad3)
- U32 pad 8: (no net) -> Net-(U28-Pad4)
- U33 pad 1: (no net) -> Net-(U29-Pad5)
- U33 pad 2: (no net) -> Net-(U29-Pad6)
- U33 pad 3: (no net) -> Net-(U29-Pad7)
- U33 pad 4: (no net) -> Net-(U29-Pad8)
- U33 pad 5: (no net) -> Net-(U33-Pad5)
- U33 pad 6: (no net) -> Net-(U33-Pad6)
- U33 pad 7: (no net) -> Net-(U33-Pad7)
- U33 pad 8: (no net) -> Net-(U33-Pad8)
- U35 pad 1: (no net) -> Net-(U35-Pad1)
- U35 pad 2: (no net) -> Net-(U35-Pad2)
- U35 pad 3: (no net) -> Net-(U35-Pad3)
- U35 pad 4: (no net) -> Net-(U35-Pad4)
- U35 pad 5: (no net) -> Net-(U32-Pad1)
- U35 pad 6: (no net) -> Net-(U32-Pad2)
- U35 pad 7: (no net) -> Net-(U32-Pad3)
- U35 pad 8: (no net) -> Net-(U32-Pad4)
- U36 pad 1: (no net) -> GND
- U36 pad 2: (no net) -> Net-(J11-Pad1)
- U36 pad 3: (no net) -> Net-(J11-Pad2)
- U36 pad 4: (no net) -> +5V
- U36 pad 5: (no net) -> Net-(U36-Pad5)
- U36 pad 6: (no net) -> Net-(U36-Pad6)
- U36 pad 7: (no net) -> Net-(U36-Pad7)
- U36 pad 8: (no net) -> Net-(U36-Pad8)
- U37 pad 1: (no net) -> Net-(U33-Pad5)
- U37 pad 2: (no net) -> Net-(U33-Pad6)
- U37 pad 3: (no net) -> Net-(U33-Pad7)
- U37 pad 4: (no net) -> Net-(U33-Pad8)
- U37 pad 5: (no net) -> Net-(U37-Pad5)
- U37 pad 6: (no net) -> Net-(U37-Pad6)
- U37 pad 7: (no net) -> Net-(U37-Pad7)
- U37 pad 8: (no net) -> Net-(U37-Pad8)
- U39 pad 1: (no net) -> Net-(U36-Pad5)
- U39 pad 2: (no net) -> Net-(U36-Pad6)
- U39 pad 3: (no net) -> Net-(U36-Pad7)
- U39 pad 4: (no net) -> Net-(U36-Pad8)
- U39 pad 5: (no net) -> Net-(U39-Pad5)
- U39 pad 6: (no net) -> Net-(U39-Pad6)
- U39 pad 7: (no net) -> Net-(U39-Pad7)
- U39 pad 8: (no net) -> Net-(U39-Pad8)
- U40 pad 1: (no net) -> Net-(U37-Pad5)
- U40 pad 2: (no net) -> Net-(U37-Pad6)
- U40 pad 3: (no net) -> Net-(U37-Pad7)
- U40 pad 4: (no net) -> Net-(U37-Pad8)
- U40 pad 5: (no net) -> Net-(U40-Pad5)
- U40 pad 6: (no net) -> Net-(U40-Pad6)
- U40 pad 7: (no net) -> Net-(U40-Pad7)
- U40 pad 8: (no net) -> Net-(U40-Pad8)
- U41 pad 6: (no net) -> Net-(J6-Pad1)
- U41 pad 7: (no net) -> Net-(J6-Pad2)
- U43 pad 1: (no net) -> Net-(U39-Pad5)
- U43 pad 2: (no net) -> Net-(U39-Pad6)
- U43 pad 3: (no net) -> Net-(U39-Pad7)
- U43 pad 4: (no net) -> Net-(U39-Pad8)
- U43 pad 5: (no net) -> Net-(U35-Pad1)
- U43 pad 6: (no net) -> Net-(U35-Pad2)
- U43 pad 7: (no net) -> Net-(U35-Pad3)
- U43 pad 8: (no net) -> Net-(U35-Pad4)
- U44 pad 1: (no net) -> Net-(U40-Pad5)
- U44 pad 2: (no net) -> Net-(U40-Pad6)
- U44 pad 3: (no net) -> Net-(U40-Pad7)
- U44 pad 4: (no net) -> Net-(U40-Pad8)
- U44 pad 5: (no net) -> Net-(U44-Pad5)
- U44 pad 6: (no net) -> Net-(U44-Pad6)
- U44 pad 7: (no net) -> Net-(U44-Pad7)
- U44 pad 8: (no net) -> Net-(U44-Pad8)
- U47 pad 1: (no net) -> Net-(U47-Pad1)
- U47 pad 2: (no net) -> Net-(U47-Pad2)
- U47 pad 3: (no net) -> Net-(U47-Pad3)
- U47 pad 4: (no net) -> Net-(U47-Pad4)
- U47 pad 5: (no net) -> Net-(U47-Pad5)
- U47 pad 6: (no net) -> Net-(U47-Pad6)
- U47 pad 7: (no net) -> Net-(U47-Pad7)
- U47 pad 8: (no net) -> Net-(U47-Pad8)
- U48 pad 1: (no net) -> Net-(U47-Pad5)
- U48 pad 2: (no net) -> Net-(U47-Pad6)
- U48 pad 3: (no net) -> Net-(U47-Pad7)
- U48 pad 4: (no net) -> Net-(U47-Pad8)
- U48 pad 5: (no net) -> Net-(U30-Pad1)
- U48 pad 6: (no net) -> Net-(U30-Pad2)
- U48 pad 7: (no net) -> Net-(U30-Pad3)
- U48 pad 8: (no net) -> Net-(U30-Pad4)
- U51 pad 1: (no net) -> Net-(U44-Pad8)
- U51 pad 2: (no net) -> Net-(U44-Pad7)
- U51 pad 3: (no net) -> Net-(U44-Pad6)
- U51 pad 4: (no net) -> Net-(U44-Pad5)
- U51 pad 5: (no net) -> Net-(U47-Pad1)
- U51 pad 6: (no net) -> Net-(U47-Pad2)
- U51 pad 7: (no net) -> Net-(U47-Pad3)
- U51 pad 8: (no net) -> Net-(U47-Pad4)
- U54 pad 1: (no net) -> GND
- U54 pad 2: (no net) -> Net-(J14-Pad1)
- U54 pad 3: (no net) -> Net-(J14-Pad2)
- U54 pad 4: (no net) -> +5V
- U68 pad 2: (no net) -> Net-(J8-Pad1)
- U68 pad 3: (no net) -> Net-(J8-Pad2)
- U71 pad 1: (no net) -> GND
- U71 pad 2: (no net) -> Net-(J16-Pad1)
- U71 pad 3: (no net) -> Net-(J16-Pad2)
- U71 pad 4: (no net) -> +5V
- U75 pad 6: (no net) -> Net-(J19-Pad1)
- U75 pad 7: (no net) -> Net-(J19-Pad2)
- U76 pad 6: (no net) -> Net-(J9-Pad1)
- U76 pad 7: (no net) -> Net-(J9-Pad2)
- U78 pad 6: (no net) -> Net-(J20-Pad1)
- U78 pad 7: (no net) -> Net-(J20-Pad2)
- U81 pad 1: (no net) -> GND
- U81 pad 2: (no net) -> Net-(J18-Pad1)
- U81 pad 3: (no net) -> Net-(J18-Pad2)
- U81 pad 4: (no net) -> +5V
- U92 pad 1: (no net) -> GND
- U92 pad 2: (no net) -> Net-(J22-Pad1)
- U92 pad 3: (no net) -> Net-(J22-Pad2)
- U92 pad 4: (no net) -> +5V
- U96 pad 6: (no net) -> Net-(J27-Pad1)
- U96 pad 7: (no net) -> Net-(J27-Pad2)
- U98 pad 1: (no net) -> GND
- U98 pad 2: (no net) -> Net-(J24-Pad1)
- U98 pad 3: (no net) -> Net-(J24-Pad2)
- U98 pad 4: (no net) -> +5V
- U98 pad 5: (no net) -> Net-(U101-Pad1)
- U98 pad 6: (no net) -> Net-(U101-Pad2)
- U98 pad 7: (no net) -> Net-(U101-Pad3)
- U98 pad 8: (no net) -> Net-(U101-Pad4)
- U99 pad 6: (no net) -> Net-(J28-Pad1)
- U99 pad 7: (no net) -> Net-(J28-Pad2)
Routing:
- net Net-(U55-Pad4): track 0.00 -> 170.5 mm, vias 0 -> 2
- net Net-(U55-Pad3): track 0.00 -> 161.9 mm, vias 0 -> 2
- net Net-(U55-Pad2): track 0.00 -> 155.2 mm, vias 0 -> 2
- net Net-(U103-Pad8): track 0.00 -> 154.7 mm, vias 0 -> 2
- net Net-(U55-Pad1): track 0.00 -> 147.9 mm, vias 0 -> 2
- net Net-(U103-Pad7): track 0.00 -> 145.4 mm, vias 0 -> 2
- net Net-(U103-Pad6): track 0.00 -> 139.0 mm, vias 0 -> 2
- net Net-(U103-Pad5): track 0.00 -> 131.8 mm, vias 0 -> 2
- net Net-(U89-Pad6): track 0.00 -> 103.0 mm
- net Net-(U89-Pad7): track 0.00 -> 103.0 mm
- net Net-(U89-Pad5): track 0.00 -> 103.0 mm
- net Net-(U89-Pad8): track 0.00 -> 103.0 mm
- net Net-(U56-Pad8): track 0.00 -> 103.0 mm
- net Net-(U56-Pad7): track 0.00 -> 103.0 mm
- net Net-(U56-Pad6): track 0.00 -> 103.0 mm
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
Commit message: finish all the tracks
Connections:
- U47 pad 1: Net-(U47-Pad1) -> Net-(U44-Pad5)
- U47 pad 2: Net-(U47-Pad2) -> Net-(U44-Pad6)
- U47 pad 3: Net-(U47-Pad3) -> Net-(U44-Pad7)
- U47 pad 4: Net-(U47-Pad4) -> Net-(U44-Pad8)
- U48 pad 1: Net-(U47-Pad5) -> Net-(U48-Pad1)
- U48 pad 2: Net-(U47-Pad6) -> Net-(U48-Pad2)
- U48 pad 3: Net-(U47-Pad7) -> Net-(U48-Pad3)
- U48 pad 4: Net-(U47-Pad8) -> Net-(U48-Pad4)
- U51 pad 1: Net-(U44-Pad8) -> Net-(U47-Pad5)
- U51 pad 2: Net-(U44-Pad7) -> Net-(U47-Pad6)
- U51 pad 3: Net-(U44-Pad6) -> Net-(U47-Pad7)
- U51 pad 4: Net-(U44-Pad5) -> Net-(U47-Pad8)
- U51 pad 5: Net-(U47-Pad1) -> Net-(U48-Pad1)
- U51 pad 6: Net-(U47-Pad2) -> Net-(U48-Pad2)
- U51 pad 7: Net-(U47-Pad3) -> Net-(U48-Pad3)
- U51 pad 8: Net-(U47-Pad4) -> Net-(U48-Pad4)
Routing:
- net Net-(U109-Pad1): track 0.00 -> 209.1 mm
- net Net-(U109-Pad2): track 0.00 -> 208.8 mm
- net Net-(U109-Pad3): track 0.00 -> 208.6 mm
- net Net-(U109-Pad4): track 0.00 -> 208.2 mm
- net Net-(U134-Pad8): track 0.00 -> 142.4 mm
- net Net-(U134-Pad7): track 0.00 -> 128.1 mm
- net Net-(U134-Pad6): track 0.00 -> 116.4 mm
- net Net-(U48-Pad1): track 0.00 -> 105.6 mm, vias 0 -> 2
- net Net-(U84-Pad5): track 0.00 -> 100.5 mm
- net Net-(U105-Pad5): track 0.00 -> 100.5 mm
- net Net-(U122-Pad8): track 0.00 -> 100.4 mm
- net Net-(U134-Pad5): track 0.00 -> 100.3 mm
- net Net-(U93-Pad8): track 0.00 -> 99.5 mm
- net Net-(U48-Pad2): track 0.00 -> 98.1 mm
- net Net-(U65-Pad5): track 0.00 -> 96.5 mm
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
Commit message: Layout done!
Parts:
- J1, J10, J13, J15, J17, J21, J23, J25, J4, J7: footprint Pin_Headers:Pin_Header_Straight_1x02_Pitch2.54mm -> connector:Power_Connector
- J11, J12, J14, J16, J18, J19, J2, J20, J22, J24, J26, J27, J28, J29, J3, J30, J5, J6, J8, J9: footprint Pin_Headers:Pin_Header_Straight_1x02_Pitch2.54mm -> connector:Sign_Connector
- moved J6 514.6 mm to (253.0, 177.0)
- moved J23 306.6 mm to (211.3, 434.6)
- moved J7 149.6 mm to (433.6, 385.1)
- moved J11 120.9 mm to (239.3, 405.1)
- moved J9 97.2 mm to (433.6, 175.3)
- moved J8 93.7 mm to (405.9, 185.9)
- moved J5 89.3 mm to (225.3, 188.2)
- moved J17 86.2 mm to (405.9, 199.4)
- moved J14 83.0 mm to (308.6, 645.2)
- moved J13 78.8 mm to (225.3, 202.4)
- moved J15 75.0 mm to (58.7, 183.1)
- moved J10 74.0 mm to (530.9, 385.8)
- moved J30 72.5 mm to (794.5, 505.7)
- moved J29 68.7 mm to (600.2, 144.5)
- moved J12 53.7 mm to (183.6, 381.3)
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Routing:
- net +5V: track 0.00 -> 395.5 mm
- net GND: track 0.00 -> 332.5 mm
- net Net-(J12-Pad1): track 0.00 -> 39.4 mm
- net Net-(J29-Pad2): track 0.00 -> 38.0 mm
- net Net-(J14-Pad2): track 0.00 -> 31.5 mm
- net Net-(J24-Pad2): track 0.00 -> 30.2 mm
- net Net-(J14-Pad1): track 0.00 -> 25.5 mm
- net Net-(J30-Pad1): track 0.00 -> 24.9 mm
- net Net-(J29-Pad1): track 0.00 -> 23.6 mm
- net Net-(J24-Pad1): track 0.00 -> 23.1 mm
- net Net-(J20-Pad1): track 0.00 -> 22.9 mm
- net Net-(J28-Pad1): track 0.00 -> 22.7 mm
- net Net-(J9-Pad1): track 0.00 -> 21.9 mm
- net Net-(J27-Pad2): track 0.00 -> 21.7 mm
- net Net-(J19-Pad2): track 0.00 -> 21.0 mm
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