File: boards/d/d.kicad_pcb (KiCad board)
At the start: 2 copper layers, 184.6 x 240.1 mm, 21 parts, among them J4 CONN_01X02, J5 CONN_01X02, J6 CONN_01X02, U31 APA102C_x5, U34 APA102C_x9, U38 APA102C_x11, U41 APA102C_x5, U42 APA102C_x3, U45 APA102C_x4, U46 APA102C_x3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

Commit message: Generate gerbers for all letters. Use a single drill size.
Other:
- net class Default: via_dia 0.6 -> None; via_drill 0.4 -> 1
- net class Signal: via_dia 0.6 -> None; via_drill 0.4 -> 1

Commit message: Boards made! Start implementing controller.
Other:
- net class Default: via_dia None -> 0.6; via_drill 1 -> 0.6
- net class Signal: via_dia None -> 0.6; via_drill 1 -> 0.6
Changed lines of the file:
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@@
   (general
     (links 74)
-    (no_connects 2)
-    (area 209.313899 35.702799 394.019401 275.963901)
+    (no_connects 0)
+    (area 12.463899 29.3277 197.169401 269.6389)
     (thickness 1.6)
     (drawings 258)
@@
       (padsonsilk false)
       (subtractmaskfromsilk false)
-      (outputformat 1)
+      (outputformat 3)
       (mirror false)
       (drillshape 0)
@@
     (clearance 0.6)
     (trace_width 2)
-    (via_drill 1)
+    (via_dia 0.6)
     (via_drill 0.6)
     (uvia_dia 0.3)
@@
     (clearance 0.6)
     (trace_width 1)
-    (via_drill 1)
+    (via_dia 0.6)
     (via_drill 0.6)
     (uvia_dia 0.3)
