File: boards/j/j.kicad_pcb (KiCad board)
At the start: 2 copper layers, 142.9 x 240.1 mm, 13 parts, among them J13 CONN_01X02, J14 CONN_01X02, J19 CONN_01X02, U54 APA102C_x3, U57 APA102C_x4, U59 APA102C_x3, U61 APA102C_x3, U63 APA102C_x4, U65 APA102C_x9, U67 APA102C_x13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

Commit message: Generate gerbers for all letters. Use a single drill size.
Other:
- net class Default: via_drill 0.4 -> 0.6
- net class Signal: via_drill 0.4 -> 0.6

Commit message: Boards made! Start implementing controller.
Parts:
- moved U65 33.9 mm to (81.3, 164.2)
- moved U69 33.9 mm to (109.1, 94.7)
- moved J13 33.9 mm to (32.8, 216.7)
- moved U54 33.9 mm to (11.9, 205.8)
- moved U57 33.9 mm to (25.7, 212.8)
- moved U59 33.9 mm to (39.6, 219.7)
- moved U63 33.9 mm to (67.4, 198.9)
- moved J14 33.9 mm to (18.8, 209.0)
- moved J19 33.9 mm to (129.8, 18.0)
- moved U61 33.9 mm to (53.5, 219.7)
- moved U67 33.9 mm to (95.2, 122.5)
- moved U75 33.9 mm to (136.9, 25.3)
- moved U72 33.9 mm to (123.0, 60.0)
