File: boards/m/m.kicad_pcb (KiCad board)
At the start: 2 copper layers, 267.9 x 170.7 mm, 26 parts, among them J25 CONN_01X02, J26 CONN_01X02, J30 CONN_01X02, U102 APA102C_x2, U105 APA102C_x5, U108 APA102C_x10, U111 APA102C_x12, U113 APA102C_x8, U115 APA102C_x3, U117 APA102C_x3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

Commit message: Generate gerbers for all letters. Use a single drill size.
Other:
- net class Default: via_drill 0.4 -> 0.6
- net class Signal: via_drill 0.4 -> 0.6

Commit message: Boards made! Start implementing controller.
Parts:
- moved U139 204.0 mm to (76.7, 24.1), turned to 0 degrees
- moved J30 188.5 mm to (86.3, 31.3), turned to 90 degrees
- moved U102 180.9 mm to (173.9, 274.1), turned to 0 degrees
- moved U134 180.9 mm to (41.9, 79.7), turned to 0 degrees
- moved U138 172.9 mm to (97.5, 38.0), turned to 180 degrees
- moved J26 169.7 mm to (167.0, 267.3), turned to 90 degrees
- moved U105 158.1 mm to (153.0, 260.3), turned to 180 degrees
- moved U119 157.6 mm to (41.9, 176.9), turned to 180 degrees
- moved U132 153.8 mm to (55.8, 93.6), turned to 180 degrees
- moved U122 153.8 mm to (41.9, 163.0), turned to 0 degrees
- moved U137 150.9 mm to (104.4, 51.9), turned to 0 degrees
- moved J25 150.1 mm to (166.8, 253.3), turned to 90 degrees
- moved U117 145.6 mm to (55.8, 190.8), turned to 0 degrees
- moved U108 145.3 mm to (118.3, 246.4), turned to 0 degrees
- moved U113 143.1 mm to (76.7, 218.6), turned to 0 degrees
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Other:
- board size 267.9 x 170.7 mm -> 170.7 x 267.9 mm
