File: boards/y/y.kicad_pcb (KiCad board)
At the start: 2 copper layers, 198.4 x 240.1 mm, 19 parts, among them J23 CONN_01X02, J24 CONN_01X02, J29 CONN_01X02, U101 APA102C_x4, U104 APA102C_x3, U106 APA102C_x2, U107 APA102C_x3, U109 APA102C_x9, U110 APA102C_x3, U112 APA102C_x16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

Commit message: Generate gerbers for all letters. Use a single drill size.
Other:
- net class Default: via_drill 0.4 -> 0.6
- net class Signal: via_drill 0.4 -> 0.6
