File: boards/all/all.kicad_pcb (KiCad board)
At the start: 2 copper layers, 767.9 x 642.9 mm, 169 parts, among them J1 CONN_01X02, J10 CONN_01X02, J11 CONN_01X02, J12 CONN_01X02, J13 CONN_01X02, J14 CONN_01X02, J15 CONN_01X02, J16 CONN_01X02, J17 CONN_01X02, J18 CONN_01X02, J19 CONN_01X02, J2 CONN_01X02, J20 CONN_01X02, J21 CONN_01X02, J22 CONN_01X02, J23 CONN_01X02, J24 CONN_01X02, J25 CONN_01X02, J26 CONN_01X02, J27 CONN_01X02, J28 CONN_01X02, J29 CONN_01X02, J3 CONN_01X02, J30 CONN_01X02, J4 CONN_01X02, J5 CONN_01X02, J6 CONN_01X02, J7 CONN_01X02, J8 CONN_01X02, J9 CONN_01X02, U1 APA102C_x6, U10 APA102C_x2, U100 APA102C_x6, U101 APA102C_x4, U102 APA102C_x2, U103 APA102C_x1, U104 APA102C_x3, U105 APA102C_x5, U106 APA102C_x2, U107 APA102C_x3, U108 APA102C_x10, U109 APA102C_x9, U11 APA102C_x2, U110 APA102C_x3, U111 APA102C_x12, U112 APA102C_x16, U113 APA102C_x8, U114 APA102C_x13, U115 APA102C_x3, U116 APA102C_x6, U117 APA102C_x3, U118 APA102C_x6, U119 APA102C_x3, U12 APA102C_x2, U120 APA102C_x2, U121 APA102C_x6, U122 APA102C_x3, U123 APA102C_x6, U124 APA102C_x7, U125 APA102C_x12, U126 APA102C_x6, U127 APA102C_x11, U128 APA102C_x4, U129 APA102C_x6, U13 APA102C_x2, U130 APA102C_x2, U131 APA102C_x2, U132 APA102C_x3, U133 APA102C_x1, U134 APA102C_x3, U135 APA102C_x3, U136 APA102C_x12, U137 APA102C_x12, U138 APA102C_x9, U139 APA102C_x4, U14 APA102C_x3, U15 APA102C_x3, U16 APA102C_x3, U17 APA102C_x3, U18 APA102C_x5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

Commit message: Generate gerbers for all letters. Use a single drill size.
Other:
- net class Default: via_dia 0.6 -> None; via_drill 0.4 -> 1
- net class Signal: via_dia 0.6 -> None; via_drill 0.4 -> 1

Commit message: Add laser cut diffuser.
Other:
- net class Default: via_dia None -> 0.6; via_drill 1 -> 0.6
- net class Signal: via_dia None -> 0.6; via_drill 1 -> 0.6
Changed lines of the file:
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@@
       (padsonsilk false)
       (subtractmaskfromsilk false)
-      (outputformat 1)
+      (outputformat 3)
       (mirror false)
       (drillshape 0)
@@
     (clearance 0.6)
     (trace_width 2)
-    (via_drill 1)
+    (via_dia 0.6)
     (via_drill 0.6)
     (uvia_dia 0.3)
@@
     (clearance 0.6)
     (trace_width 1)
-    (via_drill 1)
+    (via_dia 0.6)
     (via_drill 0.6)
     (uvia_dia 0.3)
